File: KiCAD/Owl_Cape/out-ports1-8.sch (KiCad schematic (older format))
At the start: 43 parts, among them J1 G D V, J2 G D V, J3 G D V, J4 284514-3, J5 G D V, J6 G D V, J7 G D V, J8 G D V, J9 G D V

Commit message: updates to power components
Parts:
- IC1: renamed from IC?; footprint DIP794W53P254L2540H508Q20N -> SamacSys_Parts:DIP794W53P254L2540H508Q20N
- gave numbers to parts that had none: 9
- renumbered J9 to J10, J1 to J2, J2 to J3, J3 to J4, J4 to J5, J5 to J6, J6 to J7, J7 to J8, J8 to J9, R2 to R10, R3 to R11, R4 to R12, R5 to R13, R6 to R14, R7 to R15, R8 to R16, R1 to R9

Commit message: logo and kicad updates
Parts:
- removed J10, J2, J3, J4, J6, J7, J8, J9: G D V, PhoenixContact_MCV_1,5_3-G-3.5_1x03_P3.50mm_Vertical_Tim, symbol Connector_Generic:Conn_01x03
- added J2, J3, J4, J5, J6, J7, J8: G D V, SamacSys_Parts:SHDR3W80P0X350_1X3_1250X725X940P, symbol SamacSys_Parts:284514-3
- C1: value C_Small -> 0.1uF; footprint (none) -> Capacitor_SMD:CP_Elec_4x5.3
- D1, D2, D3, D4, D5, D6, D7, D8: footprint 3544again:LED_0603_1608Metric -> LED_SMD:LED_0603_1608Metric
- F1, F2, F3, F4, F5, F6, F7, F8: footprint 3544again:3544-2 -> Fuse:Fuseholder_Blade_Mini_Keystone_3568
- J1: renamed from J5; value 284514-3 -> G D V
- R1, R2, R3, R4, R5, R6, R7, R8: footprint (none) -> Resistor_SMD:R_0805_2012Metric
- R10, R11, R12, R13, R14, R15, R16, R9: footprint 3544again:R_0805_2012Metric -> Resistor_SMD:R_0805_2012Metric
Connections:
- net GND: now also J1.1, J2.1, J3.1, J4.1, J5.1, J6.1, J7.1, J8.1
- net at D1.2 (A), F1.1: now also J1.3
- net at R1.1: now also J1.2
- net at D2.2 (A), F2.1: now also J2.3
- net at R2.1: now also J2.2
- net at D3.2 (A), F3.1: now also J3.3
- net at R3.1: now also J3.2
- net at D4.2 (A), F4.1: now also J4.3
- net at R4.1: now also J4.2
- net at D5.2 (A), F5.1: now also J5.3
- net at R5.1: now also J5.2
- net at D6.2 (A), F6.1: now also J6.3
- net at R6.1: now also J6.2
- net at D7.2 (A), F7.1: now also J7.3
- net at R7.1: now also J7.2
- net at D8.2 (A), F8.1: now also J8.3
- net at R8.1: now also J8.2
Other:
- moved on the sheet: C1, D1, D2, D3, D4, D5, D6, D7, D8, F1, F2, F3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
