File: KiCAD/Owl_Cape/power.sch (KiCad schematic (older format))
At the start: 21 parts, among them J19 VIN1_V, J20 VIN2_V, J21 Aux In, J22 9-16 In, J23 1-8 In, SW1 Enter BTN, SW2 Down BTN, U2 MP1584

Commit message: logo and kicad updates
Parts:
- removed J19: VIN1_V, Connector_JST:JST_XH_B2B-XH-A_1x02_P2.50mm_Vertical, symbol Connector:Conn_01x02_Male
- removed J20: VIN2_V, Connector_JST:JST_XH_B2B-XH-A_1x02_P2.50mm_Vertical, symbol Connector:Conn_01x02_Male
- D17, D18, D19: footprint 3544again:LED_0603_1608Metric -> LED_SMD:LED_0603_1608Metric
- F17, F18, F19: footprint 3544again:3544-2 -> Fuse:Fuseholder_Blade_Mini_Keystone_3568
- R29, R30, R31: footprint 3544again:R_0805_2012Metric -> Resistor_SMD:R_0805_2012Metric
Other:
- note added: "Buck DC-DC Step-down 12v to 5v - purchased as a seperate PCB addon"
Changed lines of the file:
@@
 encoding utf-8
 Sheet 5 5
-Title ""
+Title "The Owl - RPI Cape 16ch Pixel Controller"
 Date ""
 Rev ""
-Comp ""
+Comp "OnlineDynamic"
 Comment1 ""
 Comment2 ""
@@
 F 0 "D17" V 2539 1282 50  0000 R CNN
 F 1 "V1 LED" V 2448 1282 50  0000 R CNN
-F 2 "3544again:LED_0603_1608Metric" H 2500 1400 50  0001 C CNN
+F 2 "LED_SMD:LED_0603_1608Metric" H 2500 1400 50  0001 C CNN
 F 3 "Everlight-Elec-19-217-GHC-YR1S2-3T_C72043.pdf" H 2500 1400 50  0001 C CNN
 F 4 "C72043" H 2500 1400 50  0001 C CNN "Description"
@@
 F 0 "D18" V 2489 2882 50  0000 R CNN
 F 1 "V2 LED" V 2398 2882 50  0000 R CNN
-F 2 "3544again:LED_0603_1608Metric" H 2450 3000 50  0001 C CNN
+F 2 "LED_SMD:LED_0603_1608Metric" H 2450 3000 50  0001 C CNN
 F 3 "Everlight-Elec-19-217-GHC-YR1S2-3T_C72043.pdf" H 2450 3000 50  0001 C CNN
 F 4 "C72043" H 2450 3000 50  0001 C CNN "Description"
@@
 F 0 "R29" H 2559 1696 50  0000 L CNN
 F 1 "4.7k" H 2559 1605 50  0000 L CNN
-F 2 "3544again:R_0805_2012Metric" H 2500 1650 50  0001 C CNN
+F 2 "Resistor_SMD:R_0805_2012Metric" H 2500 1650 50  0001 C CNN
 F 3 "https://datasheet.lcsc.com/szlcsc/Uniroyal-Elec-0805W8F2201T5E_C17520.pdf" H 2500 1650 50  0001 C CNN
 F 4 "C17673" H 2500 1650 50  0001 C CNN "Description"
@@
 F 0 "R30" H 2509 2796 50  0000 L CNN
 F 1 "4.7k" H 2509 2705 50  0000 L CNN
-F 2 "3544again:R_0805_2012Metric" H 2450 2750 50  0001 C CNN
+F 2 "Resistor_SMD:R_0805_2012Metric" H 2450 2750 50  0001 C CNN
 F 3 "https://datasheet.lcsc.com/szlcsc/Uniroyal-Elec-0805W8F2201T5E_C17520.pdf" H 2450 2750 50  0001 C CNN
 F 4 "C17673" H 2450 2750 50  0001 C CNN "Description"
@@
 F 0 "R31" H 2459 3996 50  0000 L CNN
 F 1 "4.7k" H 2459 3905 50  0000 L CNN
-F 2 "3544again:R_0805_2012Metric" H 2400 3950 50  0001 C CNN
+F 2 "Resistor_SMD:R_0805_2012Metric" H 2400 3950 50  0001 C CNN
 F 3 "https://datasheet.lcsc.com/szlcsc/Uniroyal-Elec-0805W8F2201T5E_C17520.pdf" H 2400 3950 50  0001 C CNN
 F 4 "C17673" H 2400 3950 50  0001 C CNN "Description"
@@
 F 0 "D19" V 2439 4082 50  0000 R CNN
 F 1 "5V LED" V 2348 4082 50  0000 R CNN
-F 2 "3544again:LED_0603_1608Metric" H 2400 4200 50  0001 C CNN
+F 2 "LED_SMD:LED_0603_1608Metric" H 2400 4200 50  0001 C CNN
 F 3 "Everlight-Elec-19-217-GHC-YR1S2-3T_C72043.pdf" H 2400 4200 50  0001 C CNN
 F 4 "C72043" H 2400 4200 50  0001 C CNN "Description"
@@
 $EndComp
 $Comp
-L Connector:Conn_01x02_Male J19
-U 1 1 602DD954
-P 1150 1450
-F 0 "J19" V 1100 1450 50  0000 R CNN
-F 1 "VIN1_V" V 1000 1500 50  0000 R CNN
-F 2 "Connector_JST:JST_XH_B2B-XH-A_1x02_P2.50mm_Vertical" H 1150 1450 50  0001 C CNN
-F 3 "~" H 1150 1450 50  0001 C CNN
-	1    1150 1450
-	0    1    -1   0
-$EndComp
-Wire Wire Line
-	850  1150 1050 1150
-Wire Wire Line
-	1050 1150 1050 1250
-$Comp
-L Connector:Conn_01x02_Male J20
-U 1 1 602EA3C3
-P 1100 2850
-F 0 "J20" V 1050 2850 50  0000 R CNN
-F 1 "VIN2_V" V 950 2900 50  0000 R CNN
-F 2 "Connector_JST:JST_XH_B2B-XH-A_1x02_P2.50mm_Vertical" H 1100 2850 50  0001 C CNN
-F 3 "~" H 1100 2850 50  0001 C CNN
-	1    1100 2850
-	0    1    -1   0
-$EndComp
-Connection ~ 1050 1150
-Wire Wire Line
-	1150 1250 1850 1250
-$Comp
 L power:+5V #PWR058
 U 1 1 600F4BDE
@@
 F 0 "F17" V 753 3850 50  0000 C CNN
 F 1 "2A Max" V 844 3850 50  0000 C CNN
-F 2 "3544again:3544-2" V 880 3850 50  0001 C CNN
+F 2 "Fuse:Fuseholder_Blade_Mini_Keystone_3568" V 880 3850 50  0001 C CNN
 F 3 "~" H 950 3850 50  0001 C CNN
 	1    950  3850
@@
 Text GLabel 1100 3850 2    50   Input ~ 0
 V5
-Wire Wire Line
-	1100 2650 1700 2650
-Wire Wire Line
-	1000 2650 1000 2550
-Wire Wire Line
-	800  2550 1000 2550
-Connection ~ 1000 2550
-Wire Wire Line
-	1050 1150 1850 1150
-Wire Wire Line
-	1000 2550 1700 2550
-Connection ~ 1700 2650
 $Comp
 L power:GND #PWR069
@@
 	1    0    0    1
 $EndComp
-Text GLabel 6100 4150 2    50   Input ~ 0
+Text GLabel 6150 3850 2    50   Input ~ 0
 Buck
 $Comp
 L power:GND #PWR075
 U 1 1 602DB4D0
-P 6100 4350
-F 0 "#PWR075" H 6100 4100 50  0001 C CNN
-F 1 "GND" H 6105 4177 50  0000 C CNN
-F 2 "" H 6100 4350 50  0001 C CNN
-F 3 "" H 6100 4350 50  0001 C CNN
-	1    6100 4350
+P 6150 4050
+F 0 "#PWR075" H 6150 3800 50  0001 C CNN
+F 1 "GND" H 6155 3877 50  0000 C CNN
+F 2 "" H 6150 4050 50  0001 C CNN
+F 3 "" H 6150 4050 50  0001 C CNN
+	1    6150 4050
 	1    0    0    -1
 $EndComp
@@
 	0    1    1    0
 $EndComp
-Text GLabel 4800 4150 0    50   Input ~ 0
+Text GLabel 4850 3850 0    50   Input ~ 0
 Aux_In
 $Comp
 L Mirage-rescue:MP1584-MP1584 U2
 U 1 1 6057B19B
-P 5400 4250
-F 0 "U2" H 5400 4250 50  0001 L BNN
-F 1 "MP1584" H 5400 4250 50  0001 L BNN
-F 2 "DC-BRICK" H 5400 4250 50  0001 L BNN
-F 3 "" H 5400 4250 50  0001 L BNN
-	1    5400 4250
+P 5450 3950
+F 0 "U2" H 5450 3950 50  0001 L BNN
+F 1 "MP1584" H 5450 3950 50  0001 L BNN
+F 2 "DC-BRICK" H 5450 3950 50  0001 L BNN
+F 3 "" H 5450 3950 50  0001 L BNN
+	1    5450 3950
 	1    0    0    -1
 $EndComp
@@
 L power:GND #PWR072
 U 1 1 6057C09A
-P 4800 4350
-F 0 "#PWR072" H 4800 4100 50  0001 C CNN
-F 1 "GND" H 4805 4177 50  0000 C CNN
-F 2 "" H 4800 4350 50  0001 C CNN
-F 3 "" H 4800 4350 50  0001 C CNN
-	1    4800 4350
+P 4850 4050
+F 0 "#PWR072" H 4850 3800 50  0001 C CNN
+F 1 "GND" H 4855 3877 50  0000 C CNN
+F 2 "" H 4850 4050 50  0001 C CNN
+F 3 "" H 4850 4050 50  0001 C CNN
+	1    4850 4050
 	1    0    0    -1
 $EndComp
@@
 F 0 "F18" V 3353 1400 50  0000 C CNN
 F 1 "30A Max" V 3444 1400 50  0000 C CNN
-F 2 "3544again:3544-2" V 3480 1400 50  0001 C CNN
+F 2 "Fuse:Fuseholder_Blade_Mini_Keystone_3568" V 3480 1400 50  0001 C CNN
 F 3 "~" H 3550 1400 50  0001 C CNN
 	1    3550 1400
@@
 F 0 "F19" V 3303 2800 50  0000 C CNN
 F 1 "30A Max" V 3394 2800 50  0000 C CNN
-F 2 "3544again:3544-2" V 3430 2800 50  0001 C CNN
+F 2 "Fuse:Fuseholder_Blade_Mini_Keystone_3568" V 3430 2800 50  0001 C CNN
 F 3 "~" H 3500 2800 50  0001 C CNN
 	1    3500 2800
@@
 Text GLabel 3500 2950 3    50   Input ~ 0
 V2
-Connection ~ 1850 1250
 $Comp
 L Connector:Screw_Terminal_01x02 J23
@@
 Text Notes 750  2250 0    50   ~ 10
 Ports 9-16 Power
+Wire Wire Line
+	850  1150 1850 1150
+Wire Wire Line
+	800  2550 1700 2550
+Text Notes 4850 3650 0    50   ~ 10
+Buck DC-DC Step-down 12v to 5v - purchased as a seperate PCB addon
 $EndSCHEMATC
