File: KiCAD/Owl_Cape/outports9-16.kicad_sch (KiCad schematic)
At the start: 42 parts, among them IC2 SN74HC244N, J10 G D V, J11 G D V, J12 G D V, J13 G D V, J14 G D V, J15 G D V, J16 G D V, J9 G D V

Commit message: started routing cu
Changed lines of the file:
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@@
-    (stroke (width 0) (type default) (color 0 0 0 0))
-  )
-  (wire (pts (xy 90.17 85.09) (xy 90.17 87.63))
     (stroke (width 0) (type default) (color 0 0 0 0))
   )
@@
   )
   (wire (pts (xy 55.88 120.65) (xy 55.88 129.54))
+    (stroke (width 0) (type default) (color 0 0 0 0))
+  )
+  (wire (pts (xy 90.17 76.2) (xy 90.17 87.63))
     (stroke (width 0) (type default) (color 0 0 0 0))
   )
@@
     (pin "1")
   )
-  (symbol (lib_id "power:+5V") (at 90.17 85.09 0) (unit 1)
-    (in_bom yes) (on_board yes)
-    (property "Reference" "#PWR0118" (id 0) (at 90.17 88.9 0)
-      (effects (font (size 1.27 1.27)) hide)
-    )
-    (property "Value" "+5V" (id 1) (at 90.551 80.6958 0))
-    (property "Footprint" "" (id 2) (at 90.17 85.09 0)
-      (effects (font (size 1.27 1.27)) hide)
-    )
-    (property "Datasheet" "" (id 3) (at 90.17 85.09 0)
-      (effects (font (size 1.27 1.27)) hide)
-    )
+  (symbol (lib_id "power:+5V") (at 90.17 76.2 0) (unit 1)
+    (in_bom yes) (on_board yes)
+    (property "Reference" "#PWR0118" (id 0) (at 90.17 80.01 0)
+      (effects (font (size 1.27 1.27)) hide)
+    )
+    (property "Value" "+5V" (id 1) (at 90.551 71.8058 0))
+    (property "Footprint" "" (id 2) (at 90.17 76.2 0)
+      (effects (font (size 1.27 1.27)) hide)
+    )
+    (property "Datasheet" "" (id 3) (at 90.17 76.2 0)
+      (effects (font (size 1.27 1.27)) hide)
+    )
