File: KiCAD/Owl_Cape/ethernet.kicad_sch (KiCad schematic)
At the start: 6 parts, among them J18 8P8C_LED_Shielded, J19 8P8C_LED_Shielded, J20 8P8C_LED_Shielded, U4 LAN7500-ABJZ

Commit message: major update to layout
Parts:
- added IC4: KSZ8794CNXIC, QFN40P800X800X90-65N, symbol SamacSys_Parts:KSZ8794CNXIC
- J18: value 8P8C_LED_Shielded -> UPLINK
- J19: value 8P8C_LED_Shielded -> LAN 1
- J20: value 8P8C_LED_Shielded -> LAN 2
Connections:
- net GND: no longer J18.11, J18.9, J18.SH
- net at J18.1: no longer U4.43 (TR0N)
- net at J18.10: no longer U4.31 (GPIO0)
- net at J18.12: no longer U4.32 (GPIO1)
- net at J18.2: no longer U4.44 (TR0P)
- net at J18.3: no longer U4.46 (TR1N)
- net at J18.4: no longer U4.47 (TR1P)
- net at J18.5: no longer U4.51 (TR2N)
- net at J18.6: no longer U4.52 (TR2P)
- net at J18.7: no longer U4.54 (TR3N)
- net at J18.8: no longer U4.55 (TR3P)
Other:
- note added: "Ethernet 4 Port Switch"
- note added: "USB to Ethernet"
- note added: "WIP"
- company: (none) -> OnlineDynamic
- title: (none) -> The Owl - RPI Cape 16ch Pixel Controller
- moved on the sheet: J18
