File: KiCAD/Owl_Cape/owl_cape.kicad_pcb (KiCad board)
At the start: 2 copper layers, 5 parts, among them IC1 SN74LVC245AN, IC2 SN74LVC245AN, J18 Conn_02x20_Odd_Even_MountingP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, J4 284514-3

Commit message: updates to power components
Parts:
- removed J18: Conn_02x20_Odd_Even_MountingPin, Connector_PinHeader_2.54mm:PinHeader_2x20_P2.54mm_Vertical_SMD
- added D20: SB5100, Diode_THT:D_DO-201AD_P12.70mm_Horizontal, F.Cu at (226.0, 96.0)
- added D21: SB5100, Diode_THT:D_DO-201AD_P12.70mm_Horizontal, F.Cu at (226.0, 89.2)
- added D22: SB5100, Diode_THT:D_DO-201AD_P12.70mm_Horizontal, F.Cu at (243.4, 89.2)
- added D23: Zenner 5.1, Diode_THT:D_5W_P10.16mm_Horizontal, F.Cu at (225.8, 116.5)
- added H10: MountingHole, MountingHole:MountingHole_3.2mm_M3_Pad_TopBottom, F.Cu at (270.4, 104.4)
- added H5: MountingHole, MountingHole:MountingHole_3.2mm_M3_Pad_TopBottom, F.Cu at (278.3, 113.5)
- added H6: MountingHole, MountingHole:MountingHole_3.2mm_M3_Pad_TopBottom, F.Cu at (278.3, 105.6)
- added H7: MountingHole, MountingHole:MountingHole_3.2mm_M3_Pad_TopBottom, F.Cu at (278.3, 97.6)
- added H8: MountingHole, MountingHole:MountingHole_3.2mm_M3_Pad_TopBottom, F.Cu at (270.4, 112.3)
- added H9: MountingHole, MountingHole:MountingHole_3.2mm_M3_Pad_TopBottom, F.Cu at (262.4, 112.9)
- added J1: Conn_02x20_Odd_Even_MountingPin, Connector_PinHeader_2.54mm:PinHeader_2x20_P2.54mm_Vertical_SMD, F.Cu at (127.8, 112.3)
- added J19: VIN1_V, Connector_JST:JST_XH_B2B-XH-A_1x02_P2.50mm_Vertical, F.Cu at (276.8, 89.2)
- added J20: VIN2_V, Connector_JST:JST_XH_B2B-XH-A_1x02_P2.50mm_Vertical, F.Cu at (264.2, 61.0)
- added J21: Aux In, TerminalBlock_MetzConnect:TerminalBlock_MetzConnect_Type701_RT11L02HGLU_1x02_P6.35mm_Horizontal, F.Cu at (268.0, 143.5)
- added J22: 9-16 In, TerminalBlock_MetzConnect:TerminalBlock_MetzConnect_Type701_RT11L02HGLU_1x02_P6.35mm_Horizontal, F.Cu at (232.4, 149.9)
- added J23: 1-8 In, TerminalBlock_MetzConnect:TerminalBlock_MetzConnect_Type701_RT11L02HGLU_1x02_P6.35mm_Horizontal, F.Cu at (95.2, 149.9)
- added J5: 284514-3, SamacSys_Parts:SHDR3W80P0X350_1X3_1250X725X940P, F.Cu at (124.6, 148.6)
- added Q1: MMDT5401, Package_TO_SOT_SMD:SOT-363_SC-70-6, F.Cu at (234.2, 130.2)
- added Q2: DMG2302U, Package_TO_SOT_SMD:SOT-23, F.Cu at (234.3, 126.0)
- added SW1: Enter BTN, Button_Switch_THT:SW_PUSH_6mm, F.Cu at (257.9, 102.4)
- added SW2: Down BTN, Button_Switch_THT:SW_PUSH_6mm, F.Cu at (248.9, 59.7)
- added U1: AT24C256C, Package_SO:SOIC-8_3.9x4.9mm_P1.27mm, F.Cu at (227.8, 126.9)
- IC1: value SN74LVC245AN -> SN74HC244N
- J4: value 284514-3 -> G D V
Connections:
- IC1 pad 1: Net-(IC1-Pad1) -> GND
- IC1 pad 10: Net-(IC1-Pad10) -> GND
- IC1 pad 11: Net-(IC1-Pad11) -> DATA5
- IC1 pad 13: Net-(IC1-Pad13) -> DATA6
- IC1 pad 15: Net-(IC1-Pad15) -> DATA7
- IC1 pad 17: Net-(IC1-Pad17) -> DATA8
- IC1 pad 19: Net-(IC1-Pad19) -> GND
- IC1 pad 20: Net-(IC1-Pad20) -> +5V
- IC1 pad 3: DATA2 -> Net-(IC1-Pad3)
- IC1 pad 4: DATA3 -> DATA2
- IC1 pad 5: DATA4 -> Net-(IC1-Pad5)
- IC1 pad 6: DATA5 -> DATA3
- IC1 pad 7: DATA6 -> Net-(IC1-Pad7)
- IC1 pad 8: DATA7 -> DATA4
- IC1 pad 9: DATA8 -> Net-(IC1-Pad9)
- IC2 pad 10: Net-(IC2-Pad10) -> GND
- IC2 pad 20: Net-(IC2-Pad20) -> +5V
- J4 pad 1: Net-(J4-Pad1) -> GND

Commit message: logo and kicad updates
Parts:
- added H10: MountingHole, MountingHole:MountingHole_3.2mm_M3_Pad_TopBottom, F.Cu at (154.0, 84.1)
- added H5: MountingHole, MountingHole:MountingHole_3.2mm_M3_Pad_TopBottom, F.Cu at (154.0, 92.1)
- added H6: MountingHole, MountingHole:MountingHole_3.2mm_M3_Pad_TopBottom, F.Cu at (138.1, 84.1)
- added H7: MountingHole, MountingHole:MountingHole_3.2mm_M3_Pad_TopBottom, F.Cu at (138.1, 92.1)
- added H8: MountingHole, MountingHole:MountingHole_3.2mm_M3_Pad_TopBottom, F.Cu at (146.0, 84.1)
- added H9: MountingHole, MountingHole:MountingHole_3.2mm_M3_Pad_TopBottom, F.Cu at (146.0, 92.1)
- added IC2: SN74HC244N, SamacSys_Parts:DIP794W53P254L2540H508Q20N, F.Cu at (123.2, 58.2)
- added J10: G D V, SamacSys_Parts:SHDR3W80P0X350_1X3_1250X725X940P, F.Cu at (162.6, 47.8)
- added J11: G D V, SamacSys_Parts:SHDR3W80P0X350_1X3_1250X725X940P, F.Cu at (148.2, 56.8)
- added J12: G D V, SamacSys_Parts:SHDR3W80P0X350_1X3_1250X725X940P, F.Cu at (162.6, 56.8)
- added J13: G D V, SamacSys_Parts:SHDR3W80P0X350_1X3_1250X725X940P, F.Cu at (148.2, 65.7)
- added J14: G D V, SamacSys_Parts:SHDR3W80P0X350_1X3_1250X725X940P, F.Cu at (176.9, 47.8)
- added J15: G D V, SamacSys_Parts:SHDR3W80P0X350_1X3_1250X725X940P, F.Cu at (162.6, 65.7)
- added J16: G D V, SamacSys_Parts:SHDR3W80P0X350_1X3_1250X725X940P, F.Cu at (176.9, 56.8)
- added J2: G D V, SamacSys_Parts:SHDR3W80P0X350_1X3_1250X725X940P, F.Cu at (213.7, 65.7)
- added J3: G D V, SamacSys_Parts:SHDR3W80P0X350_1X3_1250X725X940P, F.Cu at (228.0, 47.8)
- added J4: G D V, SamacSys_Parts:SHDR3W80P0X350_1X3_1250X725X940P, F.Cu at (213.7, 56.8)
- added J5: G D V, SamacSys_Parts:SHDR3W80P0X350_1X3_1250X725X940P, F.Cu at (199.3, 65.7)
- added J6: G D V, SamacSys_Parts:SHDR3W80P0X350_1X3_1250X725X940P, F.Cu at (199.3, 47.8)
- added J7: G D V, SamacSys_Parts:SHDR3W80P0X350_1X3_1250X725X940P, F.Cu at (213.7, 47.8)
- added J8: G D V, SamacSys_Parts:SHDR3W80P0X350_1X3_1250X725X940P, F.Cu at (199.3, 56.8)
- added J9: G D V, SamacSys_Parts:SHDR3W80P0X350_1X3_1250X725X940P, F.Cu at (148.2, 47.8)
- J1: renamed from J5; value 284514-3 -> G D V
- moved H10 254.7 mm to (26.5, 178.0)
- moved H7 254.7 mm to (34.5, 171.3)
- moved H5 254.7 mm to (34.5, 187.2)
- moved H6 254.7 mm to (34.5, 179.2)
- moved H8 254.7 mm to (26.5, 186.0)
- moved H9 222.8 mm to (50.8, 182.9)
- moved J4 72.5 mm to (228.6, 57.1)
- moved REF** 66.6 mm to (47.0, 49.5)
- renumbered J1 to J30
Connections:
- J1 pad 1: Net-(J5-Pad1) -> GND

Commit message: added buck and pi
Parts:
- removed H10 (x2), H7 (x2), H8 (x2), H9 (x2): MountingHole, MountingHole:MountingHole_3.2mm_M3_Pad_TopBottom
- removed the H5 at (34.5, 187.2)
- removed the H6 at (34.5, 179.2)
- removed the IC2 at (203.7, 103.9)
- removed the IC2 at (123.2, 58.2)
- removed J19: VIN1_V, Connector_JST:JST_XH_B2B-XH-A_1x02_P2.50mm_Vertical
- removed J20: VIN2_V, Connector_JST:JST_XH_B2B-XH-A_1x02_P2.50mm_Vertical
- removed J21: Aux In, TerminalBlock_MetzConnect:TerminalBlock_MetzConnect_Type701_RT11L02HGLU_1x02_P6.35mm_Horizontal
- removed the J4 at (228.6, 57.1)
- removed REF**: Raspberry_Pi_Zero_Socketed_THT_FaceDown_MountingHoles, Module:Raspberry_Pi_Zero_Socketed_THT_FaceDown_MountingHoles
- added C1: 0.1uF, Capacitor_SMD:CP_Elec_4x5.3, F.Cu at (119.5, 70.7)
- added C2: 0.1uF, Capacitor_SMD:CP_Elec_4x5.3, F.Cu at (147.0, 49.2)
- added C3: 0.1uF, Capacitor_SMD:CP_Elec_4x5.3, F.Cu at (203.7, 70.2)
- added D1: 0603, LED_SMD:LED_0603_1608Metric, F.Cu at (76.6, 132.9)
- added D10: 0603, LED_SMD:LED_0603_1608Metric, F.Cu at (177.9, 132.6)
- added D11: 0603, LED_SMD:LED_0603_1608Metric, F.Cu at (189.0, 132.8)
- added D12: 0603, LED_SMD:LED_0603_1608Metric, F.Cu at (200.5, 133.0)
- added D13: 0603, LED_SMD:LED_0603_1608Metric, F.Cu at (212.2, 133.0)
- added D14: 0603, LED_SMD:LED_0603_1608Metric, F.Cu at (223.5, 133.0)
- added D15: 0603, LED_SMD:LED_0603_1608Metric, F.Cu at (234.5, 133.2)
- added D16: 0603, LED_SMD:LED_0603_1608Metric, F.Cu at (245.7, 133.0)
- added D17: V1 LED, LED_SMD:LED_0603_1608Metric, F.Cu at (65.2, 111.3)
- added D18: V2 LED, LED_SMD:LED_0603_1608Metric, F.Cu at (253.1, 111.8)
- added D19: 5V LED, LED_SMD:LED_0603_1608Metric, F.Cu at (80.2, 36.7)
- added D2: 0603, LED_SMD:LED_0603_1608Metric, F.Cu at (87.2, 132.9)
- added D3: 0603, LED_SMD:LED_0603_1608Metric, F.Cu at (99.1, 132.8)
- added D4: 0603, LED_SMD:LED_0603_1608Metric, F.Cu at (110.5, 132.9)
- added D5: 0603, LED_SMD:LED_0603_1608Metric, F.Cu at (121.7, 133.0)
- added D6: 0603, LED_SMD:LED_0603_1608Metric, F.Cu at (132.9, 132.9)
- added D7: 0603, LED_SMD:LED_0603_1608Metric, F.Cu at (144.6, 132.9)
- added D8: 0603, LED_SMD:LED_0603_1608Metric, F.Cu at (155.9, 132.8)
- added D9: 0603, LED_SMD:LED_0603_1608Metric, F.Cu at (166.2, 132.5)
- added F1: P1, Fuse:Fuseholder_Blade_Mini_Keystone_3568, F.Cu at (73.2, 127.0)
- added F10: P2, Fuse:Fuseholder_Blade_Mini_Keystone_3568, F.Cu at (175.0, 127.0)
- added F11: P3, Fuse:Fuseholder_Blade_Mini_Keystone_3568, F.Cu at (186.4, 127.0)
- added F12: P4, Fuse:Fuseholder_Blade_Mini_Keystone_3568, F.Cu at (197.7, 127.0)
- added F13: P5, Fuse:Fuseholder_Blade_Mini_Keystone_3568, F.Cu at (209.0, 127.0)
- added F14: P6, Fuse:Fuseholder_Blade_Mini_Keystone_3568, F.Cu at (220.3, 127.0)
- added F15: P7, Fuse:Fuseholder_Blade_Mini_Keystone_3568, F.Cu at (231.6, 127.0)
- added F16: P8, Fuse:Fuseholder_Blade_Mini_Keystone_3568, F.Cu at (243.0, 127.0)
- added F17: 2A Max, Fuse:Fuseholder_Blade_Mini_Keystone_3568, F.Cu at (50.3, 63.7)
- added F18: 30A Max, Fuse:Fuseholder_Blade_Mini_Keystone_3568, F.Cu at (61.8, 127.0)
- added F19: 30A Max, Fuse:Fuseholder_Blade_Mini_Keystone_3568, F.Cu at (254.0, 127.0)
- added F2: P2, Fuse:Fuseholder_Blade_Mini_Keystone_3568, F.Cu at (84.5, 127.0)
- added F3: P3, Fuse:Fuseholder_Blade_Mini_Keystone_3568, F.Cu at (95.8, 127.0)
- added F4: P4, Fuse:Fuseholder_Blade_Mini_Keystone_3568, F.Cu at (110.5, 117.1)
- added F5: P5, Fuse:Fuseholder_Blade_Mini_Keystone_3568, F.Cu at (118.4, 127.0)
- added F6: P6, Fuse:Fuseholder_Blade_Mini_Keystone_3568, F.Cu at (129.8, 127.0)
- added F7: P7, Fuse:Fuseholder_Blade_Mini_Keystone_3568, F.Cu at (141.1, 127.0)
- added F8: P8, Fuse:Fuseholder_Blade_Mini_Keystone_3568, F.Cu at (152.4, 127.0)
- added F9: P1, Fuse:Fuseholder_Blade_Mini_Keystone_3568, F.Cu at (163.7, 127.0)
- added H1: M3 MountingHole, MountingHole:MountingHole_3.2mm_M3_Pad_TopBottom, F.Cu at (46.2, 151.2)
- added H2: M3 MountingHole, MountingHole:MountingHole_3.2mm_M3_Pad_TopBottom, F.Cu at (271.0, 149.9)
- added H3: M3 MountingHole, MountingHole:MountingHole_3.2mm_M3_Pad_TopBottom, F.Cu at (271.0, 19.2)
- added H4: M3 MountingHole, MountingHole:MountingHole_3.2mm_M3_Pad_TopBottom, F.Cu at (46.3, 19.5)
- added IC2: SN74HC244N, SamacSys_Parts:DIP794W53P254L2540H508Q20N, F.Cu at (203.7, 91.3)
- added IC3: Raspberry_Pi_Zero_W__v1.3_, SamacSys_Parts:RASPBERRYPIZEROWV13, F.Cu at (158.0, 28.9)
- added J17: OLED, Connector_PinSocket_2.54mm:PinSocket_1x04_P2.54mm_Vertical, F.Cu at (197.1, 25.2)
- added R1: 4.7k, Resistor_SMD:R_0805_2012Metric, F.Cu at (72.7, 133.0)
- added R10: 4.7k, Resistor_SMD:R_0805_2012Metric, F.Cu at (174.0, 132.8)
- added R11: 4.7k, Resistor_SMD:R_0805_2012Metric, F.Cu at (185.3, 132.9)
- added R12: 4.7k, Resistor_SMD:R_0805_2012Metric, F.Cu at (196.9, 133.0)
- added R13: 4.7k, Resistor_SMD:R_0805_2012Metric, F.Cu at (208.5, 133.1)
- added R14: 4.7k, Resistor_SMD:R_0805_2012Metric, F.Cu at (219.9, 133.1)
- added R15: 4.7k, Resistor_SMD:R_0805_2012Metric, F.Cu at (230.9, 133.2)
- added R16: 4.7k, Resistor_SMD:R_0805_2012Metric, F.Cu at (242.1, 133.0)
- added R17: 33, Resistor_SMD:R_0805_2012Metric, F.Cu at (109.3, 97.2)
- added R18: 33, Resistor_SMD:R_0805_2012Metric, F.Cu at (109.4, 91.8)
- added R19: 33, Resistor_SMD:R_0805_2012Metric, F.Cu at (109.3, 87.1)
- added R2: 4.7k, Resistor_SMD:R_0805_2012Metric, F.Cu at (83.3, 132.9)
- added R20: 33, Resistor_SMD:R_0805_2012Metric, F.Cu at (109.6, 81.9)
- added R21: 33, Resistor_SMD:R_0805_2012Metric, F.Cu at (128.2, 82.4)
- added R22: 33, Resistor_SMD:R_0805_2012Metric, F.Cu at (127.4, 89.4)
- added R23: 33, Resistor_SMD:R_0805_2012Metric, F.Cu at (127.3, 94.6)
- added R24: 33, Resistor_SMD:R_0805_2012Metric, F.Cu at (128.1, 100.1)
- added R25: 33, Resistor_SMD:R_0805_2012Metric, F.Cu at (193.7, 96.7)
- added R26: 33, Resistor_SMD:R_0805_2012Metric, F.Cu at (193.8, 91.8)
- added R27: 33, Resistor_SMD:R_0805_2012Metric, F.Cu at (193.9, 86.5)
- added R28: 33, Resistor_SMD:R_0805_2012Metric, F.Cu at (194.1, 81.5)
- added R29: 33, Resistor_SMD:R_0805_2012Metric, F.Cu at (211.6, 81.1)
- added R3: 4.7k, Resistor_SMD:R_0805_2012Metric, F.Cu at (95.4, 132.9)
- added R30: 33, Resistor_SMD:R_0805_2012Metric, F.Cu at (211.5, 86.1)
- added R31: 33, Resistor_SMD:R_0805_2012Metric, F.Cu at (212.0, 90.8)
- added R32: 33, Resistor_SMD:R_0805_2012Metric, F.Cu at (211.5, 96.1)
- added R33: 4.7k, Resistor_SMD:R_0805_2012Metric, F.Cu at (165.6, 51.0)
- added R34: 4.7k, Resistor_SMD:R_0805_2012Metric, F.Cu at (165.7, 47.3)
- added R35: 10k, Resistor_SMD:R_0805_2012Metric, F.Cu at (109.6, 17.7)
- added R36: 4.7k, Resistor_SMD:R_0805_2012Metric, F.Cu at (115.5, 16.3)
- added R37: 4.7k, Resistor_SMD:R_0805_2012Metric, F.Cu at (61.3, 111.3)
- added R38: 4.7k, Resistor_SMD:R_0805_2012Metric, F.Cu at (257.4, 111.9)
- added R39: 4.7k, Resistor_SMD:R_0805_2012Metric, F.Cu at (88.9, 38.1)
- added R4: 4.7k, Resistor_SMD:R_0805_2012Metric, F.Cu at (106.7, 133.0)
- added R5: 4.7k, Resistor_SMD:R_0805_2012Metric, F.Cu at (118.0, 133.1)
- added R6: 4.7k, Resistor_SMD:R_0805_2012Metric, F.Cu at (129.1, 133.0)
- added R7: 4.7k, Resistor_SMD:R_0805_2012Metric, F.Cu at (140.9, 132.9)
- added R8: 4.7k, Resistor_SMD:R_0805_2012Metric, F.Cu at (152.1, 132.8)
- added R9: 4.7k, Resistor_SMD:R_0805_2012Metric, F.Cu at (162.4, 132.7)
- added U2: D-SUN_MP1584_BUCK, Stuart_BESPOKE:D-SUN_MP1584_BUCK, F.Cu at (60.6, 71.8)
- H5, H6: value MountingHole -> M3 MountingHole
- J22, J23: footprint TerminalBlock_MetzConnect:TerminalBlock_MetzConnect_Type701_RT11L02HGLU_1x02_P6.35mm_Horizontal -> TerminalBlock_MetzConnect:TerminalBlock_MetzConnect_Type703_RT10N02HGLU_1x02_P9.52mm_Horizontal
- J30: footprint Connector_PinHeader_2.54mm:PinHeader_2x20_P2.54mm_Vertical_SMD -> Connector_PinHeader_2.54mm:PinHeader_2x20_P2.54mm_Vertical
- moved D23 198.7 mm to (46.1, 31.7)
- moved D22 174.9 mm to (75.3, 41.0), turned to 180 degrees
- moved D20 173.4 mm to (52.7, 103.0)
- moved J3 166.7 mm to (88.9, 139.7)
- moved J2 162.5 mm to (76.2, 152.4)
- moved Q1 159.9 mm to (111.5, 27.6)
- moved Q2 158.0 mm to (115.8, 21.5)
- moved J4 147.3 mm to (101.6, 152.4)
- moved J6 127.2 mm to (127.0, 152.4)
- moved J16 122.8 mm to (254.0, 152.4)
- moved J7 118.0 mm to (139.7, 139.7)
- moved J14 116.7 mm to (228.6, 152.4)
- moved H5 116.3 mm to (92.1, 190.5)
- moved H6 115.1 mm to (73.6, 179.5)
- moved J5 112.7 mm to (114.3, 139.7)
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Connections:
- IC1 pad 20: +5V -> V5Rail
- J30 pad 13: Net-(J30-Pad13) -> unconnected-(J30-Pad13)
- J30 pad 18: Net-(J30-Pad18) -> BTN1
- J30 pad 22: Net-(J30-Pad22) -> BTN2
- J30 pad 26: Net-(J30-Pad26) -> unconnected-(J30-Pad26)
- J30 pad 29: Net-(J30-Pad29) -> unconnected-(J30-Pad29)
- J30 pad 3: Net-(J30-Pad3) -> unconnected-(J30-Pad3)
- J30 pad 31: Net-(J30-Pad31) -> unconnected-(J30-Pad31)
- J30 pad 37: Net-(J30-Pad37) -> unconnected-(J30-Pad37)
- J30 pad 5: Net-(J30-Pad5) -> unconnected-(J30-Pad5)
- J30 pad 7: Net-(J30-Pad7) -> unconnected-(J30-Pad7)
Other:
- board outline added: 241.5 x 146.9 mm
- net class Default removed

Commit message: started routing cu
Parts:
- added J18: 8P8C_LED_Shielded, Connector_RJ:RJ45_BEL_SS74301-00x_Vertical, F.Cu at (90.2, 28.2)
- added J19: 8P8C_LED_Shielded, Connector_RJ:RJ45_BEL_SS74301-00x_Vertical, F.Cu at (112.6, 28.2)
- added U3: TZT_Original_0.96_inch_oled_IIC_Serial_OLED_Display_Module_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, Stuart_BESPOKE:TZT_0.96inch_OLED, F.Cu at (203.0, 17.7)
- IC3: footprint SamacSys_Parts:RASPBERRYPIZEROWV13 -> Stuart_BESPOKE:RASPBERRYPIZERO2WV1
- J22: value 9-16 In -> J9-16 +12V DC In
- J23: value 1-8 In -> Cape + J1-8 +12V DC In
- moved H6 120.8 mm to (191.3, 152.4)
- moved F18 42.5 mm to (82.4, 89.8), turned to -90 degrees
- moved Q2 42.4 mm to (92.1, 56.6)
- moved Q1 42.4 mm to (87.8, 62.8)
- moved R35 42.4 mm to (85.9, 52.8)
- moved R36 42.4 mm to (91.8, 51.4)
- moved F19 35.9 mm to (251.0, 91.2), turned to -90 degrees
- moved IC3 34.3 mm to (190.3, 17.2)
- moved J22 27.1 mm to (266.6, 99.9)
- moved J23 26.5 mm to (58.1, 88.8)
- moved D17 20.7 mm to (72.4, 91.8), turned to 180 degrees
- moved R37 20.7 mm to (68.5, 91.8)
- moved F17 18.0 mm to (52.7, 45.8), turned to 0 degrees
- moved U2 16.6 mm to (65.8, 56.0)
- moved D16 16.3 mm to (262.0, 132.9), turned to 180 degrees
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Connections:
- C1 pad 1: V5Rail -> +5V
- F17 pad 2: V5Rail -> +5V
- IC1 pad 20: V5Rail -> +5V
- U2 pad 5: unconnected-(U2-Pad5) -> GND1
Routing:
- net GND: track 0.00 -> 545.7 mm
- net VIN2: track 0.00 -> 191.5 mm
- net VIN1: track 0.00 -> 48.0 mm
- net Net-(F16-Pad1): track 0.00 -> 34.2 mm
- net V1: track 0.00 -> 25.4 mm
- net Net-(F14-Pad1): track 0.00 -> 25.3 mm
- net V2: track 0.00 -> 19.4 mm
- net Net-(F15-Pad1): track 0.00 -> 15.9 mm
- net Net-(F13-Pad1): track 0.00 -> 13.9 mm
- net Net-(D18-Pad2): track 0.00 -> 3.45 mm
- net Net-(D16-Pad2): track 0.00 -> 1.98 mm
Other:
- board size 241.5 x 146.9 mm -> 232 x 146 mm

Commit message: swap chips to better speed / layout
Parts:
- removed R17, R18, R19, R20, R21, R22, R25, R26, R27, R28, R29, R30, R31, R32: 33, Resistor_SMD:R_0805_2012Metric
- added J20: 8P8C_LED_Shielded, Connector_RJ:RJ45_BEL_SS74301-00x_Vertical, F.Cu at (129.4, 20.1)
- added RN1: 33R, Resistor_THT:R_Array_SIP8, F.Cu at (75.4, 109.8)
- added RN2: 33R, Resistor_THT:R_Array_SIP8, F.Cu at (126.7, 110.0)
- added RN3: 33R, Resistor_THT:R_Array_SIP8, F.Cu at (175.9, 109.5)
- added RN4: 33R, Resistor_THT:R_Array_SIP8, F.Cu at (221.4, 109.9)
- added U4: LAN7500-ABJZ, Package_DFN_QFN:QFN-56-1EP_8x8mm_P0.5mm_EP5.9x5.9mm, F.Cu at (109.5, 47.9)
- F1: footprint Fuse:Fuseholder_Blade_Mini_Keystone_3568 -> Stuart_BESPOKE:Medium Auto Fuse Holder
- IC1: value SN74HC244N -> SN74AHC245N
- IC3: value Raspberry_Pi_Zero_W__v1.3_ -> Raspberry_Pi_Zero_2_W__v1.0_
- J22: value J9-16 +12V DC In -> 9-16 In
- J23: value Cape + J1-8 +12V DC In -> 1-8 In
- R23: value 33 -> 12k
- R24: value 33 -> 8.06K
- moved R24 82.5 mm to (146.0, 19.6)
- moved R23 80.2 mm to (146.0, 16.7)
- moved IC3 28.2 mm to (193.3, 45.1)
- moved C1 21.7 mm to (100.2, 80.6)
- moved J30 16.5 mm to (186.7, 81.3)
- moved F1 15.7 mm to (67.4, 113.8), turned to -90 degrees
- moved C3 14.2 mm to (218.9, 70.7)
- moved IC1 10.9 mm to (109.3, 95.9), turned to -90 degrees
- moved R1 10.1 mm to (59.9, 122.7), turned to -90 degrees
- moved IC2 7.45 mm to (210.3, 94.7)
- moved D1 6.50 mm to (60.0, 126.6), turned to -90 degrees
Connections:
- IC1 pad 11: DATA5 -> Net-(IC1-Pad11)
- IC1 pad 13: DATA6 -> Net-(IC1-Pad13)
- IC1 pad 15: DATA7 -> Net-(IC1-Pad15)
- IC1 pad 17: DATA8 -> Net-(IC1-Pad17)
- IC1 pad 2: DATA1 -> DATA8
- IC1 pad 3: Net-(IC1-Pad3) -> DATA7
- IC1 pad 4: DATA2 -> DATA6
- IC1 pad 5: Net-(IC1-Pad5) -> DATA5
- IC1 pad 6: DATA3 -> DATA4
- IC1 pad 7: Net-(IC1-Pad7) -> DATA3
- IC1 pad 8: DATA4 -> DATA2
- IC1 pad 9: Net-(IC1-Pad9) -> DATA1
- IC3 pad 48: unconnected-(IC3-Pad48) -> USBDP
- IC3 pad 49: unconnected-(IC3-Pad49) -> USBDM
- J18 pad 1: unconnected-(J18-Pad1) -> Net-(J18-Pad1)
- J18 pad 10: unconnected-(J18-Pad10) -> Net-(J18-Pad10)
- J18 pad 11: unconnected-(J18-Pad11) -> GND
- J18 pad 12: unconnected-(J18-Pad12) -> Net-(J18-Pad12)
- J18 pad 2: unconnected-(J18-Pad2) -> Net-(J18-Pad2)
- J18 pad 3: unconnected-(J18-Pad3) -> Net-(J18-Pad3)
- J18 pad 4: unconnected-(J18-Pad4) -> Net-(J18-Pad4)
- J18 pad 5: unconnected-(J18-Pad5) -> Net-(J18-Pad5)
- J18 pad 6: unconnected-(J18-Pad6) -> Net-(J18-Pad6)
- J18 pad 7: unconnected-(J18-Pad7) -> Net-(J18-Pad7)
- J18 pad 8: unconnected-(J18-Pad8) -> Net-(J18-Pad8)
- J18 pad 9: unconnected-(J18-Pad9) -> GND
- J19 pad SH: GND -> unconnected-(J19-PadSH)
- R23 pad 1: Net-(J7-Pad2) -> GND
- R23 pad 2: Net-(IC1-Pad5) -> Net-(R23-Pad2)
- R24 pad 1: Net-(J8-Pad2) -> GND
- R24 pad 2: Net-(IC1-Pad3) -> Net-(R24-Pad2)

Commit message: major update to layout
Parts:
- removed D22: SB5100, Diode_THT:D_DO-201AD_P12.70mm_Horizontal
- removed H5, H6: M3 MountingHole, MountingHole:MountingHole_3.2mm_M3_Pad_TopBottom
- removed SW1: Enter BTN, Button_Switch_THT:SW_PUSH_6mm
- added C4: 0.1uF, Capacitor_THT:C_Rect_L7.0mm_W2.0mm_P5.00mm, F.Cu at (183.1, 54.9)
- added IC4: KSZ8794CNXIC, SamacSys_Parts:QFN40P800X800X90-65N, F.Cu at (77.2, 67.7)
- added J21: GPIO TRG, Connector_JST:JST_XH_B3B-XH-A_1x03_P2.50mm_Vertical, F.Cu at (51.5, 58.0)
- added J24: DMX1 RJ45, Connector_RJ:RJ45_Amphenol_54602-x08_Horizontal, F.Cu at (199.0, 42.3)
- added R17: Pull_Up_resistor, Resistor_SMD:R_0805_2012Metric, F.Cu at (215.3, 89.3)
- added R18: 2.2K, Resistor_SMD:R_0805_2012Metric, F.Cu at (221.4, 92.6)
- added R19: 2.2K, Resistor_SMD:R_0805_2012Metric, F.Cu at (226.7, 92.6)
- added R20: 2.2K, Resistor_SMD:R_0805_2012Metric, F.Cu at (231.3, 92.6)
- added R21: 2.2K, Resistor_SMD:R_0805_2012Metric, F.Cu at (236.0, 92.7)
- added R22: 2.2K, Resistor_SMD:R_0805_2012Metric, F.Cu at (240.6, 92.7)
- added R25: 120, Resistor_THT:R_Axial_DIN0207_L6.3mm_D2.5mm_P7.62mm_Horizontal, F.Cu at (182.9, 44.9)
- added SW3: SW_UP, Button_Switch_THT:SW_PUSH_6mm, F.Cu at (224.6, 62.6)
- added SW4: SW_RIGHT, Button_Switch_THT:SW_PUSH_6mm, F.Cu at (236.3, 71.9)
- added SW5: SW_DOWN, Button_Switch_THT:SW_PUSH_6mm, F.Cu at (224.1, 82.1)
- added SW6: SW_LEFT, Button_Switch_THT:SW_PUSH_6mm, F.Cu at (213.0, 71.8)
- added SW7: SW_ENTER, Button_Switch_THT:SW_PUSH_6mm, F.Cu at (224.3, 71.9)
- added U5: UA9638CP, Package_DIP:DIP-8_W7.62mm, F.Cu at (170.5, 41.7)
- F10: value P2 -> P1; footprint Fuse:Fuseholder_Blade_Mini_Keystone_3568 -> Stuart_BESPOKE:Medium Auto Fuse Holder
- F11: value P3 -> P1; footprint Fuse:Fuseholder_Blade_Mini_Keystone_3568 -> Stuart_BESPOKE:Medium Auto Fuse Holder
- F12: value P4 -> P1; footprint Fuse:Fuseholder_Blade_Mini_Keystone_3568 -> Stuart_BESPOKE:Medium Auto Fuse Holder
- F13: value P5 -> P1; footprint Fuse:Fuseholder_Blade_Mini_Keystone_3568 -> Stuart_BESPOKE:Medium Auto Fuse Holder
- F14: value P6 -> P1; footprint Fuse:Fuseholder_Blade_Mini_Keystone_3568 -> Stuart_BESPOKE:Medium Auto Fuse Holder
- F15: value P7 -> P1; footprint Fuse:Fuseholder_Blade_Mini_Keystone_3568 -> Stuart_BESPOKE:Medium Auto Fuse Holder
- F16: value P8 -> P1; footprint Fuse:Fuseholder_Blade_Mini_Keystone_3568 -> Stuart_BESPOKE:Medium Auto Fuse Holder
- F17, F18, F19, F2, F3, F4, F5, F6, F7, F8, F9: footprint Fuse:Fuseholder_Blade_Mini_Keystone_3568 -> Stuart_BESPOKE:Medium Auto Fuse Holder
- IC2: value SN74HC244N -> SN74AHC245N
- J18: value 8P8C_LED_Shielded -> UPLINK
- J19: value 8P8C_LED_Shielded -> LAN 1
- J20: value 8P8C_LED_Shielded -> LAN 2
- SW2: value Down BTN -> DMX_LOR_Select; footprint Button_Switch_THT:SW_PUSH_6mm -> Button_Switch_THT:SW_CuK_JS202011CQN_DPDT_Straight
- moved R23 75.5 mm to (88.1, 65.1)
- moved R24 75.5 mm to (88.1, 68.0)
- moved C2 70.6 mm to (84.6, 83.5)
- moved R33 70.6 mm to (103.3, 85.3)
- moved R34 70.6 mm to (103.3, 81.6)
- moved U1 70.6 mm to (95.0, 84.1)
- moved F19 64.1 mm to (225.3, 150.0), turned to 90 degrees
- moved F18 63.2 mm to (62.9, 150.0), turned to 90 degrees
- moved D17 54.8 mm to (56.7, 144.3), turned to 0 degrees
- moved R39 53.7 mm to (51.5, 80.5)
- moved R37 53.1 mm to (60.6, 144.3), turned to 180 degrees
- moved U3 47.1 mm to (185.2, 61.3)
- moved J16 44.4 mm to (213.3, 127.9)
- moved F17 44.3 mm to (66.0, 88.1), turned to 180 degrees
- moved D19 43.2 mm to (60.1, 80.5)
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Connections:
- F1 pad 1: Net-(F1-Pad1) -> VIN1
- F1 pad 3: (no net) -> Net-(F1-Pad3)
- F1 pad 4: (no net) -> Net-(F1-Pad3)
- F10 pad 1: Net-(F10-Pad1) -> VIN2
- F11 pad 1: Net-(F11-Pad1) -> VIN2
- F12 pad 1: Net-(F12-Pad1) -> VIN2
- F13 pad 1: Net-(F13-Pad1) -> VIN2
- F14 pad 1: Net-(F14-Pad1) -> VIN2
- F15 pad 1: Net-(F15-Pad1) -> VIN2
- F16 pad 1: Net-(F16-Pad1) -> VIN2
- F17 pad 2: +5V -> V5
- F18 pad 2: VIN1 -> V1
- F19 pad 2: VIN2 -> V2
- F2 pad 1: Net-(F2-Pad1) -> VIN1
- F3 pad 1: Net-(F3-Pad1) -> VIN1
- F4 pad 1: Net-(F4-Pad1) -> VIN1
- F5 pad 1: Net-(F5-Pad1) -> VIN1
- F6 pad 1: Net-(F6-Pad1) -> VIN1
- F7 pad 1: Net-(F7-Pad1) -> VIN1
- F8 pad 1: Net-(F8-Pad1) -> VIN1
- F9 pad 1: Net-(F9-Pad1) -> VIN2
- IC1 pad 1: GND -> +5V
- IC2 pad 1: GND -> +5V
- IC2 pad 11: DATA13 -> Net-(IC2-Pad11)
- IC2 pad 13: DATA14 -> Net-(IC2-Pad13)
- IC2 pad 15: DATA15 -> Net-(IC2-Pad15)
- IC2 pad 17: DATA16 -> Net-(IC2-Pad17)
- IC2 pad 2: DATA9 -> DATA16
- IC2 pad 3: Net-(IC2-Pad3) -> DATA15
- IC2 pad 4: DATA10 -> DATA14
- IC2 pad 5: Net-(IC2-Pad5) -> DATA13
- IC2 pad 6: DATA11 -> DATA12
- IC2 pad 7: Net-(IC2-Pad7) -> DATA11
- IC2 pad 8: DATA12 -> DATA10
- IC2 pad 9: Net-(IC2-Pad9) -> DATA9
- J1 pad 3: Net-(F1-Pad1) -> Net-(F1-Pad3)
- J10 pad 3: Net-(F10-Pad1) -> Net-(F10-Pad3)
- J11 pad 3: Net-(F11-Pad1) -> Net-(F11-Pad3)
- J12 pad 3: Net-(F12-Pad1) -> Net-(F12-Pad3)
- J13 pad 3: Net-(F13-Pad1) -> Net-(F13-Pad3)
- J14 pad 3: Net-(F14-Pad1) -> Net-(F14-Pad3)
- J15 pad 3: Net-(F15-Pad1) -> Net-(F15-Pad3)
- J16 pad 3: Net-(F16-Pad1) -> Net-(F16-Pad3)
- J18 pad 1: Net-(J18-Pad1) -> unconnected-(J18-Pad1)
- J18 pad 10: Net-(J18-Pad10) -> unconnected-(J18-Pad10)
- J18 pad 11: GND -> unconnected-(J18-Pad11)
- J18 pad 12: Net-(J18-Pad12) -> unconnected-(J18-Pad12)
- J18 pad 2: Net-(J18-Pad2) -> unconnected-(J18-Pad2)
- J18 pad 3: Net-(J18-Pad3) -> unconnected-(J18-Pad3)
- J18 pad 4: Net-(J18-Pad4) -> unconnected-(J18-Pad4)
- J18 pad 5: Net-(J18-Pad5) -> unconnected-(J18-Pad5)
- J18 pad 6: Net-(J18-Pad6) -> unconnected-(J18-Pad6)
- J18 pad 7: Net-(J18-Pad7) -> unconnected-(J18-Pad7)
- J18 pad 8: Net-(J18-Pad8) -> unconnected-(J18-Pad8)
- J18 pad 9: GND -> unconnected-(J18-Pad9)
- J18 pad SH: GND -> unconnected-(J18-PadSH)
- J2 pad 3: Net-(F2-Pad1) -> Net-(F2-Pad3)
- J3 pad 3: Net-(F3-Pad1) -> Net-(F3-Pad3)
- J30 pad 18: BTN1 -> DATA7
- J30 pad 22: BTN2 -> BTN1
- J30 pad 29: unconnected-(J30-Pad29) -> BTN_ARRAY_ANALOGUE_IN
- J30 pad 8: DATA7 -> TXD1
- J4 pad 3: Net-(F4-Pad1) -> Net-(F4-Pad3)
- J5 pad 3: Net-(F5-Pad1) -> Net-(F5-Pad3)
- J6 pad 3: Net-(F6-Pad1) -> Net-(F6-Pad3)
- J7 pad 3: Net-(F7-Pad1) -> Net-(F7-Pad3)
- J8 pad 3: Net-(F8-Pad1) -> Net-(F8-Pad3)
- J9 pad 3: Net-(F9-Pad1) -> Net-(F9-Pad3)
- R1 pad 1: Net-(F1-Pad1) -> Net-(F1-Pad3)
- R10 pad 1: Net-(F10-Pad1) -> Net-(F10-Pad3)
- R11 pad 1: Net-(F11-Pad1) -> Net-(F11-Pad3)
- R12 pad 1: Net-(F12-Pad1) -> Net-(F12-Pad3)
- R13 pad 1: Net-(F13-Pad1) -> Net-(F13-Pad3)
- R14 pad 1: Net-(F14-Pad1) -> Net-(F14-Pad3)
- R15 pad 1: Net-(F15-Pad1) -> Net-(F15-Pad3)
- R16 pad 1: Net-(F16-Pad1) -> Net-(F16-Pad3)
- R2 pad 1: Net-(F2-Pad1) -> Net-(F2-Pad3)
- R3 pad 1: Net-(F3-Pad1) -> Net-(F3-Pad3)
- R4 pad 1: Net-(F4-Pad1) -> Net-(F4-Pad3)
- R5 pad 1: Net-(F5-Pad1) -> Net-(F5-Pad3)
- R6 pad 1: Net-(F6-Pad1) -> Net-(F6-Pad3)
- R7 pad 1: Net-(F7-Pad1) -> Net-(F7-Pad3)
- R8 pad 1: Net-(F8-Pad1) -> Net-(F8-Pad3)
- R9 pad 1: Net-(F9-Pad1) -> Net-(F9-Pad3)
- RN3 pad 1: Net-(IC2-Pad18) -> Net-(IC2-Pad11)
- RN3 pad 3: Net-(IC2-Pad16) -> Net-(IC2-Pad12)
- RN3 pad 5: Net-(IC2-Pad14) -> Net-(IC2-Pad13)
- RN3 pad 7: Net-(IC2-Pad12) -> Net-(IC2-Pad14)
- RN4 pad 1: Net-(IC2-Pad9) -> Net-(IC2-Pad15)
- RN4 pad 3: Net-(IC2-Pad7) -> Net-(IC2-Pad16)
- RN4 pad 5: Net-(IC2-Pad5) -> Net-(IC2-Pad17)
- RN4 pad 7: Net-(IC2-Pad3) -> Net-(IC2-Pad18)
- SW2 pad 1: GND -> Net-(J24-Pad4)
- SW2 pad 2: BTN2 -> /Serial_Diffs/DMX1+
- U4 pad 31: Net-(J18-Pad10) -> unconnected-(U4-Pad31)
- U4 pad 32: Net-(J18-Pad12) -> unconnected-(U4-Pad32)
- U4 pad 43: Net-(J18-Pad1) -> unconnected-(U4-Pad43)
- U4 pad 44: Net-(J18-Pad2) -> unconnected-(U4-Pad44)
- U4 pad 46: Net-(J18-Pad3) -> unconnected-(U4-Pad46)
- U4 pad 47: Net-(J18-Pad4) -> unconnected-(U4-Pad47)
- U4 pad 51: Net-(J18-Pad5) -> unconnected-(U4-Pad51)
- U4 pad 52: Net-(J18-Pad6) -> unconnected-(U4-Pad52)
- U4 pad 54: Net-(J18-Pad7) -> unconnected-(U4-Pad54)
- U4 pad 55: Net-(J18-Pad8) -> unconnected-(U4-Pad55)
Routing:
- net GND: track 545.7 -> 0.00 mm
- net VIN2: track 191.5 -> 0.00 mm
- net VIN1: track 48.0 -> 0.00 mm
- net Net-(F16-Pad1): track 34.2 -> 0.00 mm
- net V1: track 25.4 -> 0.00 mm
- net Net-(F14-Pad1): track 25.3 -> 0.00 mm
- net V2: track 19.4 -> 0.00 mm
- net Net-(F15-Pad1): track 15.9 -> 0.00 mm
- net Net-(F13-Pad1): track 13.9 -> 0.00 mm
- net Net-(D18-Pad2): track 3.45 -> 0.00 mm
- net Net-(D16-Pad2): track 1.98 -> 0.00 mm
Other:
- board size 232 x 146 mm -> 200 x 120 mm
- board text added: "JLCJLCJLCJLC"
