File: KiCAD/Owl_Cape/owl_cape.kicad_sch (KiCad schematic)
At the start: 2 parts, among them IC3 Raspberry_Pi_Zero_2_W__v1.0_, J30 Conn_02x20_Odd_Even_MountingP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

Commit message: major update to layout
Connections:
- net BTN2 is gone; now on net BTN1: J30.22 (Pin_22)
- net BTN1: no longer J30.18 (Pin_18)
- net DATA7: now also J30.18 (Pin_18); no longer J30.8 (Pin_8)
- net BTN_ARRAY_ANALOGUE_IN: now reaches J30.29 (Pin_29)
- new net TXD1: J30.8 (Pin_8)
- no-connect marks 8 -> 7
Other:
- note added: "Need to check and test pinout with anaologue in on pin 29 (GPIO5)"

Commit message: formatting fix
Connections:
- net I2C_SCL: now also J30.5 (Pin_5); no longer J30.28 (Pin_28)
- net I2C_SDA: now also J30.3 (Pin_3); no longer J30.27 (Pin_27)
- net BTN_ARRAY_ADC_IN: now reaches J30.7 (Pin_7)
- net BTN_ARRAY_ANALOGUE_IN: no longer names the net of J30.29 (Pin_29)
- new net I2C_EEPROM_SCL: J30.28 (Pin_28)
- new net I2C_EEPROM_SDA: J30.27 (Pin_27)
- no-connect marks 7 -> 5
Other:
- note added: "Need to check and test pinout with analogue in on pin 29 (GPIO5)"
- note removed: "Need to check and test pinout with anaologue in on pin 29 (GPIO5)"
Changed lines of the file:
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@@
   )
   (no_connect (at 40.64 76.2))
-  (no_connect (at 40.64 43.18))
-  (no_connect (at 40.64 45.72))
+  (no_connect (at 40.64 73.66))
   (no_connect (at 53.34 68.58))
-  (no_connect (at 40.64 40.64))
   (no_connect (at 40.64 83.82))
   (no_connect (at 40.64 53.34))
@@
     (stroke (width 0) (type default) (color 0 0 0 0))
   )
-  (wire (pts (xy 38.862 73.66) (xy 40.64 73.66))
+  (wire (pts (xy 53.34 50.8) (xy 59.69 50.8))
     (stroke (width 0) (type default) (color 0 0 0 0))
   )
-  (wire (pts (xy 53.34 50.8) (xy 59.69 50.8))
+  (wire (pts (xy 37.592 40.64) (xy 40.64 40.64))
     (stroke (width 0) (type default) (color 0 0 0 0))
   )
@@
     (stroke (width 0) (type default) (color 0 0 0 0))
   )
+  (wire (pts (xy 37.592 43.18) (xy 40.64 43.18))
+    (stroke (width 0) (type default) (color 0 0 0 0))
+  )
   (wire (pts (xy 57.15 76.2) (xy 53.34 76.2))
     (stroke (width 0) (type default) (color 0 0 0 0))
@@
     (stroke (width 0) (type default) (color 0 0 0 0))
   )
+  (wire (pts (xy 37.592 71.12) (xy 40.64 71.12))
+    (stroke (width 0) (type default) (color 0 0 0 0))
+  )
+  (wire (pts (xy 53.34 71.12) (xy 57.15 71.12))
+    (stroke (width 0) (type default) (color 0 0 0 0))
+  )
   (wire (pts (xy 36.83 60.96) (xy 40.64 60.96))
     (stroke (width 0) (type default) (color 0 0 0 0))
@@
     (stroke (width 0) (type default) (color 0 0 0 0))
   )
+  (wire (pts (xy 38.354 45.72) (xy 40.64 45.72))
+    (stroke (width 0) (type default) (color 0 0 0 0))
+  )
   (image (at 264.16 130.81)
     (data
@@
   )
   (text "Owl Cape" (at 220.98 157.48 0)
-    (effects (font (size 8.001 8.001) (thickness 1.6002) bold italic) (justify left bottom))
+    (effects (font (size 8.001 8.001) italic) (justify left bottom))
   )
   (text "40Pin RPI Header Input (via ribbon cable)" (at 22.86 26.67 0)
     (effects (font (size 1.27 1.27) (thickness 0.254) bold) (justify left bottom))
   )
-  (text "Need to check and test pinout with anaologue in on pin 29 (GPIO5)"
+  (text "Need to check and test pinout with analogue in on pin 29 (GPIO5)"
     (at 18.034 96.266 0)
     (effects (font (size 4 4) (thickness 0.8) bold) (justify left bottom))
@@
     )
   )
-  (global_label "I2C_SDA" (shape bidirectional) (at 40.64 71.12 180) (fields_autoplaced)
+  (global_label "I2C_SDA" (shape bidirectional) (at 37.592 40.64 180) (fields_autoplaced)
     (effects (font (size 1.27 1.27)) (justify right))
-    (property "Intersheet References" "${INTERSHEET_REFS}" (id 0) (at 30.6958 71.0406 0)
+    (property "Intersheet References" "${INTERSHEET_REFS}" (id 0) (at 27.6478 40.5606 0)
       (effects (font (size 1.27 1.27)) (justify right) hide)
     )
@@
     )
   )
+  (global_label "I2C_EEPROM_SDA" (shape bidirectional) (at 37.592 71.12 180) (fields_autoplaced)
+    (effects (font (size 1.27 1.27)) (justify right))
+    (property "Intersheet References" "${INTERSHEET_REFS}" (id 0) (at 19.0602 71.0406 0)
+      (effects (font (size 1.27 1.27)) (justify right) hide)
+    )
+  )
   (global_label "BTN1" (shape input) (at 59.69 63.5 0) (fields_autoplaced)
     (effects (font (size 1.27 1.27)) (justify left))
@@
     )
   )
-  (global_label "I2C_SCL" (shape bidirectional) (at 53.34 71.12 0) (fields_autoplaced)
-    (effects (font (size 1.27 1.27)) (justify left))
-    (property "Intersheet References" "${INTERSHEET_REFS}" (id 0) (at 63.2237 71.0406 0)
-      (effects (font (size 1.27 1.27)) (justify left) hide)
+  (global_label "I2C_SCL" (shape bidirectional) (at 37.592 43.18 180) (fields_autoplaced)
+    (effects (font (size 1.27 1.27)) (justify right))
+    (property "Intersheet References" "${INTERSHEET_REFS}" (id 0) (at 27.7083 43.1006 0)
+      (effects (font (size 1.27 1.27)) (justify right) hide)
     )
   )
@@
     )
   )
+  (global_label "I2C_EEPROM_SCL" (shape bidirectional) (at 57.15 71.12 0) (fields_autoplaced)
+    (effects (font (size 1.27 1.27)) (justify left))
+    (property "Intersheet References" "${INTERSHEET_REFS}" (id 0) (at 75.6213 71.0406 0)
+      (effects (font (size 1.27 1.27)) (justify left) hide)
+    )
+  )
   (global_label "DATA1" (shape output) (at 60.96 66.04 0) (fields_autoplaced)
     (effects (font (size 1.27 1.27)) (justify left))
@@
     )
   )
-  (global_label "BTN_ARRAY_ANALOGUE_IN" (shape input) (at 38.862 73.66 180) (fields_autoplaced)
+  (global_label "BTN_ARRAY_ADC_IN" (shape input) (at 38.354 45.72 180) (fields_autoplaced)
     (effects (font (size 1.27 1.27)) (justify right))
-    (property "Intersheet References" "${INTERSHEET_REFS}" (id 0) (at 12.7102 73.5806 0)
+    (property "Intersheet References" "${INTERSHEET_REFS}" (id 0) (at 18.1893 45.6406 0)
       (effects (font (size 1.27 1.27)) (justify right) hide)
     )
