File: KiCAD/Owl_Cape/serial_diff.kicad_sch (KiCad schematic)
At the start: 0 parts

Commit message: major update to layout
Parts:
- added C4: 0.1uF, Capacitor_THT:C_Rect_L7.0mm_W2.0mm_P5.00mm, symbol PB_16-rescue:C-Device
- added J24: DMX1 RJ45, Connector_RJ:RJ45_Amphenol_54602-x08_Horizontal, symbol Connector:RJ45
- added R25: 120, Resistor_THT:R_Axial_DIN0207_L6.3mm_D2.5mm_P7.62mm_Horizontal, symbol PB_16-rescue:R-Device
- added SW2: DMX_LOR_Select, Button_Switch_THT:SW_CuK_JS202011CQN_DPDT_Straight, symbol Switch:SW_DPDT_x2
- added U5: (no value), symbol Interface_LineDriver:UA9638CP
Connections:
- new net: J24.4, SW2.1 (A)
- new net: J24.1, SW2.3 (C)
- new net: J24.5, SW2.4 (A)
- new net: J24.2, SW2.6 (C)
- new net +5V: C4.1, U5.1 (VCC)
- new net 9V: J24.3
- new net DMX1+: R25.1, SW2.2 (B), U5.8 (OUTB)
- new net DMX1-: R25.2, SW2.5 (B), U5.7 (OUTA)
- new net GND: C4.2, J24.6, J24.7, J24.8, U5.4 (GND)
- new net TXD1: U5.2 (IN)
- no-connect marks 0 -> 3
Other:
- note added: "DMX1"
- company: (none) -> OnlineDynamic
- title: (none) -> The Owl - RPI Cape 16ch Pixel Controller

Commit message: formatting fix
Parts:
- U5: value (none) -> UA9638CP; footprint (none) -> Package_DIP:DIP-8_W7.62mm
Changed lines of the file:
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@@
       (effects (font (size 1.27 1.27)) (justify right))
     )
-    (property "Value" "" (id 1) (at 186.182 94.488 0)
+    (property "Value" "UA9638CP" (id 1) (at 186.182 94.488 0)
       (effects (font (size 1.27 1.27)) (justify right))
     )
-    (property "Footprint" "" (id 2) (at 170.942 113.03 0)
+    (property "Footprint" "Package_DIP:DIP-8_W7.62mm" (id 2) (at 170.942 113.03 0)
       (effects (font (size 1.27 1.27)) hide)
     )
@@
       (effects (font (size 1.27 1.27)) (justify right))
     )
-    (property "Value" "" (id 1) (at 187.071 53.594 0)
+    (property "Value" "UA9638CP" (id 1) (at 187.071 53.594 0)
       (effects (font (size 1.27 1.27)) (justify right))
     )
-    (property "Footprint" "" (id 2) (at 171.831 72.136 0)
+    (property "Footprint" "Package_DIP:DIP-8_W7.62mm" (id 2) (at 171.831 72.136 0)
       (effects (font (size 1.27 1.27)) hide)
     )
