File: KiCAD/Owl_Cape/standard-hat-components.kicad_sch (KiCad schematic)
At the start: 14 parts, among them Q1 MMDT5401, Q2 DMG2302U, U1 AT24C256C

Commit message: major update to layout
Parts:
- removed H5, H6: M3 MountingHole, MountingHole:MountingHole_3.2mm_M3_Pad_TopBottom, symbol Mechanical:MountingHole
Other:
- moved on the sheet: C2, R34, U1

Commit message: formatting fix
Connections:
- net I2C_SCL renamed I2C_EEPROM_SCL
- net I2C_SDA renamed I2C_EEPROM_SDA
Changed lines of the file:
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@@
     (stroke (width 0) (type default) (color 0 0 0 0))
   )
-  (polyline (pts (xy 80.01 62.23) (xy 80.01 101.6))
+  (polyline (pts (xy 87.884 62.23) (xy 87.884 101.6))
     (stroke (width 0) (type default) (color 0 0 0 0))
   )
@@
     (stroke (width 0) (type default) (color 0 0 0 0))
   )
-  (polyline (pts (xy 80.01 101.6) (xy 30.48 101.6))
+  (polyline (pts (xy 87.884 101.6) (xy 30.48 101.6))
     (stroke (width 0) (type default) (color 0 0 0 0))
   )
@@
     (stroke (width 0) (type default) (color 0 0 0 0))
   )
-  (polyline (pts (xy 29.21 62.23) (xy 80.01 62.23))
+  (polyline (pts (xy 29.21 62.23) (xy 87.884 62.23))
     (stroke (width 0) (type default) (color 0 0 0 0))
   )
@@
     (effects (font (size 1.524 1.524)) (justify left bottom))
   )
-  (global_label "I2C_SCL" (shape input) (at 68.58 85.09 0) (fields_autoplaced)
+  (global_label "I2C_EEPROM_SCL" (shape input) (at 68.58 85.09 0) (fields_autoplaced)
     (effects (font (size 1.27 1.27)) (justify left))
-    (property "Intersheet References" "${INTERSHEET_REFS}" (id 0) (at 3.81 8.89 0)
-      (effects (font (size 1.27 1.27)) hide)
+    (property "Intersheet References" "${INTERSHEET_REFS}" (id 0) (at 87.0513 85.0106 0)
+      (effects (font (size 1.27 1.27)) (justify left) hide)
     )
   )
-  (global_label "I2C_SDA" (shape input) (at 68.58 82.55 0) (fields_autoplaced)
+  (global_label "I2C_EEPROM_SDA" (shape input) (at 68.58 82.55 0) (fields_autoplaced)
     (effects (font (size 1.27 1.27)) (justify left))
-    (property "Intersheet References" "${INTERSHEET_REFS}" (id 0) (at 3.81 8.89 0)
-      (effects (font (size 1.27 1.27)) hide)
+    (property "Intersheet References" "${INTERSHEET_REFS}" (id 0) (at 87.1118 82.4706 0)
+      (effects (font (size 1.27 1.27)) (justify left) hide)
     )
   )

Commit message: updates based on testing
Parts:
- removed C2: 0.1uF, Capacitor_SMD:CP_Elec_4x5.3, symbol Device:C_Small
Changed lines of the file:
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@@
     (company "OnlineDynamic")
   )
-  (junction (at 48.26 77.47) (diameter 0) (color 0 0 0 0)
-  )
-  (junction (at 38.1 82.55) (diameter 0) (color 0 0 0 0)
-  )
   (junction (at 38.1 87.63) (diameter 0) (color 0 0 0 0)
   )
@@
     (stroke (width 0) (type default) (color 0 0 0 0))
   )
-  (wire (pts (xy 38.1 77.47) (xy 38.1 82.55))
-    (stroke (width 0) (type default) (color 0 0 0 0))
-  )
   (wire (pts (xy 66.04 85.09) (xy 68.58 85.09))
     (stroke (width 0) (type default) (color 0 0 0 0))
@@
   )
   (wire (pts (xy 158.75 63.5) (xy 158.75 72.39))
-    (stroke (width 0) (type default) (color 0 0 0 0))
-  )
-  (wire (pts (xy 43.18 77.47) (xy 48.26 77.47))
     (stroke (width 0) (type default) (color 0 0 0 0))
   )
@@
     (pin "1")
   )
-  (symbol (lib_id "Device:C_Small") (at 40.64 77.47 270) (unit 1)
-    (in_bom yes) (on_board yes)
-    (property "Reference" "C2" (id 0) (at 40.64 71.6534 90))
-    (property "Value" "0.1uF" (id 1) (at 40.64 73.9648 90))
-    (property "Footprint" "Capacitor_SMD:CP_Elec_4x5.3" (id 2) (at 40.64 77.47 0)
-      (effects (font (size 1.27 1.27)) hide)
-    )
-    (property "Datasheet" "https://datasheet.lcsc.com/szlcsc/Samsung-Electro-Mechanics-CL05B104KO5NNNC_C1525.pdf" (id 3) (at 40.64 77.47 0)
-      (effects (font (size 1.27 1.27)) hide)
-    )
-    (property "Description" "C49678" (id 4) (at 40.64 77.47 0)
-      (effects (font (size 1.27 1.27)) hide)
-    )
-    (pin "1")
-    (pin "2")
-  )
   (symbol (lib_id "Device:R_Small") (at 66.04 74.93 0) (unit 1)
