File: KiCAD/DPI-24/DPI-24-Controller/controls.kicad_sch (KiCad schematic)
At the start: 2 parts

Commit message: layout updates
Parts:
- added J33: GPIO TRG, Connector_JST:JST_XH_B3B-XH-A_1x03_P2.50mm_Vertical, symbol Connector:Conn_01x03_Male
- added R30: Pull_Up_resistor, Resistor_SMD:R_0805_2012Metric, symbol Device:R
- added R31, R32, R33, R34, R40: 2.2K, Resistor_SMD:R_0805_2012Metric, symbol Device:R
- added SW1: SW_UP, Button_Switch_THT:SW_PUSH_6mm, symbol Switch:SW_Push
- added SW2, SW3, SW4: (no value), Button_Switch_THT:SW_PUSH_6mm, symbol Switch:SW_Push
- added SW5: SW_ENTER, Button_Switch_THT:SW_PUSH_6mm, symbol Switch:SW_Push
- J32: value (none) -> OLED; footprint (none) -> Connector_PinSocket_2.54mm:PinSocket_1x04_P2.54mm_Vertical
- U3: value (none) -> TZT_Original_0.96_inch_oled_IIC_Serial_OLED_Display_Module_128X64; footprint (none) -> Stuart_BESPOKE:TZT_0.96inch_OLED
Connections:
- net GND: now also J33.2 (Pin_2), J33.3 (Pin_3), SW1.2, SW2.2, SW3.2, SW4.2, SW5.2
- new net: R31.2, R32.1, SW1.1
- new net: R32.2, R33.1, SW2.1
- new net: R34.2, R40.1, SW4.1
- new net: R33.2, R34.1, SW3.1
- new net: R40.2, SW5.1
- new net +5V: R30.1
- new net BTN1: J33.1 (Pin_1)
- new net SW_ARRAY_ANALOGUE_IN: R30.2, R31.1
Other:
- note added: "Control Switch Buttons"
- note added: "GENERAL GPIO Trigger Jumper"
- title: The Owl - RPI Cape 16ch Pixel Controller -> RPI Cape DPI 24ch Pixel Controller
