File: KiCAD/DPI-24/DPI-24-Controller/controls.kicad_sch (KiCad schematic)
At the start: 14 parts, among them J32 OLED, J33 GPIO TRG, SW1 UP, SW2 DOWN, SW3 BACK, SW4 TEST, SW5 ENTER, U3 TZT_Original_0.96_inch_oled_I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

Commit message: more layout tweaking and a bit of copper!
Parts:
- added C5: 0.1uF, Capacitor_THT:C_Radial_D5.0mm_H11.0mm_P2.00mm, symbol Device:C_Small
- added U5: (no value), symbol Analog_ADC:ADS1113IDGS
- J33: value GPIO TRG -> (none); footprint Connector_JST:JST_XH_B3B-XH-A_1x03_P2.50mm_Vertical -> (none)
Connections:
- net +5V: now also C5.1, U5.8 (VDD)
- net GND: now also C5.2, U5.1 (ADDR), U5.3 (GND)
- net I2C_SCL: now also U5.10 (SCL)
- net I2C_SDA: now also U5.9 (SDA)
- net SW_ARRAY_ANALOGUE_IN: now also U5.4 (AIN0)
- no-connect marks 4 -> 5
Other:
- note added: "Excluded from Board currently as no spare GPIO to connect to"
Changed lines of the file:
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@@
   (junction (at 28.702 87.63) (diameter 0) (color 0 0 0 0)
   )
-  (junction (at 28.702 84.836) (diameter 0) (color 0 0 0 0)
-  )
   (junction (at 52.832 146.05) (diameter 0) (color 0 0 0 0)
   )
@@
   (junction (at 28.702 133.35) (diameter 0) (color 0 0 0 0)
   )
+  (junction (at 127 87.63) (diameter 0) (color 0 0 0 0)
+  )
+  (no_connect (at 116.84 103.886))
   (no_connect (at 43.18 33.02))
   (no_connect (at 43.18 27.94))
@@
     (stroke (width 0) (type default) (color 0 0 0 0))
   )
+  (wire (pts (xy 127 86.106) (xy 127 87.63))
+    (stroke (width 0) (type default) (color 0 0 0 0))
+  )
   (wire (pts (xy 52.832 120.65) (xy 52.832 133.35))
     (stroke (width 0) (type default) (color 0 0 0 0))
@@
     (stroke (width 0) (type default) (color 0 0 0 0))
   )
-  (wire (pts (xy 28.702 87.63) (xy 28.702 84.836))
+  (wire (pts (xy 28.702 82.55) (xy 28.702 87.63))
     (stroke (width 0) (type default) (color 0 0 0 0))
   )
@@
     (stroke (width 0) (type default) (color 0 0 0 0))
   )
+  (wire (pts (xy 127 87.63) (xy 127 91.186))
+    (stroke (width 0) (type default) (color 0 0 0 0))
+  )
   (wire (pts (xy 160.02 39.624) (xy 157.48 42.926))
     (stroke (width 0) (type default) (color 0 0 0 0))
@@
     (stroke (width 0) (type default) (color 0 0 0 0))
   )
+  (wire (pts (xy 144.018 87.63) (xy 144.018 93.98))
+    (stroke (width 0) (type default) (color 0 0 0 0))
+  )
   (wire (pts (xy 28.702 133.35) (xy 37.592 133.35))
     (stroke (width 0) (type default) (color 0 0 0 0))
@@
     (stroke (width 0) (type default) (color 0 0 0 0))
   )
+  (wire (pts (xy 137.668 87.63) (xy 144.018 87.63))
+    (stroke (width 0) (type default) (color 0 0 0 0))
+  )
   (wire (pts (xy 28.702 87.63) (xy 36.322 87.63))
     (stroke (width 0) (type default) (color 0 0 0 0))
@@
     (stroke (width 0) (type default) (color 0 0 0 0))
   )
-  (wire (pts (xy 28.702 84.836) (xy 36.322 84.836))
-    (stroke (width 0) (type default) (color 0 0 0 0))
-  )
   (wire (pts (xy 52.832 97.79) (xy 52.832 109.22))
     (stroke (width 0) (type default) (color 0 0 0 0))
@@
     (stroke (width 0) (type default) (color 0 0 0 0))
   )
+  (wire (pts (xy 132.588 87.63) (xy 127 87.63))
+    (stroke (width 0) (type default) (color 0 0 0 0))
+  )
   (wire (pts (xy 52.832 109.22) (xy 52.832 120.65))
     (stroke (width 0) (type default) (color 0 0 0 0))
@@
     (stroke (width 0) (type default) (color 0 0 0 0))
   )
-  (wire (pts (xy 28.702 84.836) (xy 28.702 82.55))
-    (stroke (width 0) (type default) (color 0 0 0 0))
-  )
-  (text "GENERAL GPIO Trigger Jumper" (at 149.86 31.496 0)
+  (text "Excluded from Board currently as no spare GPIO to connect to"
+    (at 138.43 50.546 0)
+    (effects (font (size 1.27 1.27)) (justify left bottom))
+  )
+  (text "GENERAL GPIO Trigger Jumper" (at 148.082 21.59 0)
     (effects (font (size 1.27 1.27)) (justify left bottom))
   )
@@
   (text "Control Switch Buttons" (at 42.672 77.47 0)
     (effects (font (size 1.27 1.27)) (justify left bottom))
+  )
+  (global_label "SW_ARRAY_ANALOGUE_IN" (shape input) (at 116.84 101.346 180) (fields_autoplaced)
+    (effects (font (size 1.27 1.27)) (justify right))
+    (property "Intersheet References" "${INTERSHEET_REFS}" (id 0) (at 91.5953 101.2666 0)
+      (effects (font (size 1.27 1.27)) (justify right) hide)
+    )
   )
   (global_label "BTN1" (shape input) (at 162.56 39.624 0) (fields_autoplaced)
@@
     )
   )
-  (global_label "SW_ARRAY_GPIO_TRIGGER" (shape output) (at 36.322 84.836 0) (fields_autoplaced)
+  (global_label "I2C_SCL" (shape input) (at 137.16 103.886 0) (fields_autoplaced)
     (effects (font (size 1.27 1.27)) (justify left))
-    (property "Intersheet References" "${INTERSHEET_REFS}" (id 0) (at 62.2924 84.7566 0)
+    (property "Intersheet References" "${INTERSHEET_REFS}" (id 0) (at 147.0437 103.8066 0)
       (effects (font (size 1.27 1.27)) (justify left) hide)
     )
@@
     )
   )
+  (global_label "I2C_SDA" (shape input) (at 137.16 106.426 0) (fields_autoplaced)
+    (effects (font (size 1.27 1.27)) (justify left))
+    (property "Intersheet References" "${INTERSHEET_REFS}" (id 0) (at 147.1042 106.3466 0)
+      (effects (font (size 1.27 1.27)) (justify left) hide)
+    )
+  )
   (symbol (lib_id "Connector:Conn_01x04_Female") (at 34.29 34.29 0) (unit 1)
     (in_bom yes) (on_board yes)
@@
     (pin "3")
     (pin "4")
+  )
+  (symbol (lib_id "Device:C_Small") (at 135.128 87.63 90) (unit 1)
+    (in_bom yes) (on_board yes)
+    (property "Reference" "C5" (id 0) (at 136.906 85.344 90))
+    (property "Value" "0.1uF" (id 1) (at 135.128 91.1352 90))
+    (property "Footprint" "Capacitor_THT:C_Radial_D5.0mm_H11.0mm_P2.00mm" (id 2) (at 135.128 87.63 0)
+      (effects (font (size 1.27 1.27)) hide)
+    )
+    (property "Datasheet" "~" (id 3) (at 135.128 87.63 0)
+      (effects (font (size 1.27 1.27)) hide)
+    )
+    (pin "1")
+    (pin "2")
+  )
+  (symbol (lib_id "power:GND") (at 144.018 93.98 0) (unit 1)
+    (in_bom yes) (on_board yes) (fields_autoplaced)
+    (property "Reference" "#PWR0161" (id 0) (at 144.018 100.33 0)
+      (effects (font (size 1.27 1.27)) hide)
+    )
+    (property "Value" "GND" (id 1) (at 144.018 98.4234 0))
+    (property "Footprint" "" (id 2) (at 144.018 93.98 0)
+      (effects (font (size 1.27 1.27)) hide)
+    )
+    (property "Datasheet" "" (id 3) (at 144.018 93.98 0)
+      (effects (font (size 1.27 1.27)) hide)
+    )
+    (pin "1")
   )
   (symbol (lib_id "Device:R") (at 28.702 93.98 0) (unit 1)
@@
   )
   (symbol (lib_id "Connector:Conn_01x03_Male") (at 160.02 34.544 270) (unit 1)
-    (in_bom yes) (on_board yes)
+    (in_bom yes) (on_board no)
     (property "Reference" "J33" (id 0) (at 157.7848 35.7124 90)
       (effects (font (size 1.27 1.27)) (justify right))
     )
-    (property "Value" "GPIO TRG" (id 1) (at 157.7848 33.401 90)
+    (property "Value" "" (id 1) (at 157.7848 33.401 90)
       (effects (font (size 1.27 1.27)) (justify right))
     )
-    (property "Footprint" "Connector_JST:JST_XH_B3B-XH-A_1x03_P2.50mm_Vertical" (id 2) (at 160.02 34.544 0)
+    (property "Footprint" "" (id 2) (at 160.02 34.544 0)
       (effects (font (size 1.27 1.27)) hide)
     )
@@
     (pin "2")
     (pin "3")
+  )
+  (symbol (lib_id "power:GND") (at 127 114.046 0) (unit 1)
+    (in_bom yes) (on_board yes) (fields_autoplaced)
+    (property "Reference" "#PWR0162" (id 0) (at 127 120.396 0)
+      (effects (font (size 1.27 1.27)) hide)
+    )
+    (property "Value" "" (id 1) (at 127 118.4894 0))
+    (property "Footprint" "" (id 2) (at 127 114.046 0)
+      (effects (font (size 1.27 1.27)) hide)
+    )
+    (property "Datasheet" "" (id 3) (at 127 114.046 0)
+      (effects (font (size 1.27 1.27)) hide)
+    )
+    (pin "1")
   )
   (symbol (lib_id "Switch:SW_Push") (at 42.672 97.79 0) (unit 1)
@@
     (pin "2")
   )
+  (symbol (lib_id "power:+5V") (at 127 86.106 0) (unit 1)
+    (in_bom yes) (on_board yes) (fields_autoplaced)
+    (property "Reference" "#PWR0164" (id 0) (at 127 89.916 0)
+      (effects (font (size 1.27 1.27)) hide)
+    )
+    (property "Value" "" (id 1) (at 127 82.5302 0))
+    (property "Footprint" "" (id 2) (at 127 86.106 0)
+      (effects (font (size 1.27 1.27)) hide)
+    )
+    (property "Datasheet" "" (id 3) (at 127 86.106 0)
+      (effects (font (size 1.27 1.27)) hide)
+    )
+    (pin "1")
+  )
   (symbol (lib_id "power:+3.3V") (at 29.21 36.83 90) (unit 1)
     (in_bom yes) (on_board yes)
@@
     (pin "2")
   )
+  (symbol (lib_id "power:GND") (at 137.16 108.966 0) (unit 1)
+    (in_bom yes) (on_board yes) (fields_autoplaced)
+    (property "Reference" "#PWR0163" (id 0) (at 137.16 115.316 0)
+      (effects (font (size 1.27 1.27)) hide)
+    )
+    (property "Value" "GND" (id 1) (at 137.16 113.4094 0))
+    (property "Footprint" "" (id 2) (at 137.16 108.966 0)
+      (effects (font (size 1.27 1.27)) hide)
+    )
+    (property "Datasheet" "" (id 3) (at 137.16 108.966 0)
+      (effects (font (size 1.27 1.27)) hide)
+    )
+    (pin "1")
+  )
+  (symbol (lib_id "Analog_ADC:ADS1113IDGS") (at 127 103.886 0) (unit 1)
+    (in_bom yes) (on_board yes) (fields_autoplaced)
+    (property "Reference" "U5" (id 0) (at 129.0194 90.0262 0)
+      (effects (font (size 1.27 1.27)) (justify left))
+    )
+    (property "Value" "" (id 1) (at 129.0194 92.5631 0)
+      (effects (font (size 1.27 1.27)) (justify left))
+    )
+    (property "Footprint" "" (id 2) (at 127 116.586 0)
+      (effects (font (size 1.27 1.27)) hide)
+    )
+    (property "Datasheet" "http://www.ti.com/lit/ds/symlink/ads1113.pdf" (id 3) (at 128.27 121.666 0)
+      (effects (font (size 1.27 1.27)) hide)
+    )
+    (pin "1")
+    (pin "10")
+    (pin "2")
+    (pin "3")
+    (pin "4")
+    (pin "5")
+    (pin "6")
+    (pin "7")
+    (pin "8")
+    (pin "9")
+  )
   (symbol (lib_id "Device:R") (at 28.702 129.54 0) (unit 1)
