File: KiCAD/DPI-24/DPI-24-Controller/outports17-24.kicad_sch (KiCad schematic)
At the start: 36 parts

Commit message: layout updates
Parts:
- C4: value (none) -> 0.1uF; footprint (none) -> Capacitor_THT:C_Radial_D5.0mm_H11.0mm_P2.00mm
- D17, D18, D19, D20, D21, D22, D23, D24: value (none) -> 0603; footprint (none) -> LED_SMD:LED_0603_1608Metric
- F17, F18, F19, F20, F21, F22, F23, F24: value (none) -> P1; footprint (none) -> Stuart_BESPOKE:Medium Auto Fuse Holder
- IC3: value (none) -> SN74AHC245N; footprint (none) -> DIP794W53P254L2540H508Q20N
- J17, J18, J19, J20, J21, J22, J23, J24: value (none) -> G D V; footprint (none) -> Connector_Phoenix_MC:PhoenixContact_MCV_1,5_3-G-3.5_1x03_P3.50mm_Vertical
- R17, R18, R19, R20, R21, R22, R23, R24: value (none) -> 4.7k; footprint (none) -> Resistor_SMD:R_0805_2012Metric
- RN5, RN6: value (none) -> 33R; footprint (none) -> Resistor_THT:R_Array_SIP8
Other:
- title: The Owl - RPI Cape 16ch Pixel Controller -> RPI Cape DPI 24ch Pixel Controller
