File: KiCAD/DPI-24/DPI-24-Controller/power.kicad_sch (KiCad schematic)
At the start: 20 parts

Commit message: layout updates
Parts:
- D25: value (none) -> V1 LED; footprint (none) -> LED_SMD:LED_0603_1608Metric
- D26, D28, D30: value (none) -> SB5100; footprint (none) -> Diode_THT:D_DO-201AD_P12.70mm_Horizontal
- D27: value (none) -> V2 LED; footprint (none) -> LED_SMD:LED_0603_1608Metric
- D29: value (none) -> V3 LED; footprint (none) -> LED_SMD:LED_0603_1608Metric
- D31: value (none) -> 5V LED; footprint (none) -> LED_SMD:LED_0603_1608Metric
- D32: value (none) -> Zenner 5.1; footprint (none) -> Diode_THT:D_5W_P10.16mm_Horizontal
- F25, F26, F27: value (none) -> 30A Max; footprint (none) -> Stuart_BESPOKE:Medium Auto Fuse Holder
- F28: value (none) -> 2A Max; footprint (none) -> Stuart_BESPOKE:Medium Auto Fuse Holder
- J28: value (none) -> 1-8 In; footprint (none) -> TerminalBlock_MetzConnect:TerminalBlock_MetzConnect_Type703_RT10N02HGLU_1x02_P9.52mm_Horizontal
- J29: value (none) -> 9-16 In; footprint (none) -> TerminalBlock_MetzConnect:TerminalBlock_MetzConnect_Type703_RT10N02HGLU_1x02_P9.52mm_Horizontal
- J30: value (none) -> 17-24 In; footprint (none) -> TerminalBlock_MetzConnect:TerminalBlock_MetzConnect_Type703_RT10N02HGLU_1x02_P9.52mm_Horizontal
- R26, R37, R38, R39: value (none) -> 4.7k; footprint (none) -> Resistor_SMD:R_0805_2012Metric
- U2: value (none) -> D-SUN_MP1584_BUCK; footprint (none) -> Stuart_BESPOKE:D-SUN_MP1584_BUCK
Other:
- title: The Owl - RPI Cape 16ch Pixel Controller -> RPI Cape DPI 24ch Pixel Controller
