File: KiCAD/DPI-24/DPI-24-Controller/power.kicad_sch (KiCad schematic)
At the start: 20 parts, among them J28 Ports 1-8 12V DC IN, J29 Ports 9-16 12V DC IN, J30 Ports 17-24 12V DC IN, U2 D-SUN_MP1584_BUCK

Commit message: more layout tweaking and a bit of copper!
Parts:
- added J34: Select Voltage, Connector_PinHeader_2.54mm:PinHeader_1x03_P2.54mm_Vertical, symbol Connector_Generic:Conn_01x03
- added J35: Select Control Feed, Connector_PinHeader_2.54mm:PinHeader_1x03_P2.54mm_Vertical, symbol Connector_Generic:Conn_01x03
- added J36: Aux In, TerminalBlock_RND:TerminalBlock_RND_205-00012_1x02_P5.00mm_Horizontal, symbol Connector:Screw_Terminal_01x02
Connections:
- net GND: now also U2.2 (IN2-), J36.1 (Pin_1)
- net GND1: now also U2.6 (OUT2-)
- net V5: now also U2.8 (OUT2+), J34.1 (Pin_1)
- net VIN1: now also J35.3 (Pin_3); no longer U2.3 (IN1+)
- net BUCK_In: now reaches U2.4 (IN2+)
- net BUCK_In: now also U2.3 (IN1+), J34.3 (Pin_3)
- new net Aux_In: J35.1 (Pin_1), J36.2 (Pin_2)
- new net Control_In: J34.2 (Pin_2), J35.2 (Pin_2)
- no-connect marks 4 -> 0
Changed lines of the file:
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@@
     (company "OnlineDynamic")
   )
+  (junction (at 41.148 156.464) (diameter 0) (color 0 0 0 0)
+  )
+  (junction (at 71.628 164.084) (diameter 0) (color 0 0 0 0)
+  )
+  (junction (at 71.628 156.464) (diameter 0) (color 0 0 0 0)
+  )
   (junction (at 126.492 106.172) (diameter 0) (color 0 0 0 0)
   )
+  (junction (at 40.386 164.084) (diameter 0) (color 0 0 0 0)
+  )
   (junction (at 37.338 164.084) (diameter 0) (color 0 0 0 0)
   )
-  (no_connect (at 41.148 159.004))
-  (no_connect (at 71.628 159.004))
-  (no_connect (at 71.628 166.624))
-  (no_connect (at 41.148 166.624))
   (polyline (pts (xy 261.112 98.806) (xy 261.366 129.032))
     (stroke (width 0) (type default) (color 0 0 0 0))
@@
     (stroke (width 0) (type default) (color 0 0 0 0))
   )
+  (wire (pts (xy 71.628 164.084) (xy 71.628 166.624))
+    (stroke (width 0) (type default) (color 0 0 0 0))
+  )
   (wire (pts (xy 251.206 107.442) (xy 247.396 107.442))
     (stroke (width 0) (type default) (color 0 0 0 0))
@@
     (stroke (width 0) (type default) (color 0 0 0 0))
   )
-  (wire (pts (xy 37.338 164.084) (xy 41.148 164.084))
+  (wire (pts (xy 37.338 164.084) (xy 40.386 164.084))
     (stroke (width 0) (type default) (color 0 0 0 0))
   )
@@
     (stroke (width 0) (type default) (color 0 0 0 0))
   )
+  (wire (pts (xy 41.148 156.464) (xy 41.148 159.004))
+    (stroke (width 0) (type default) (color 0 0 0 0))
+  )
+  (wire (pts (xy 71.628 156.464) (xy 71.628 159.004))
+    (stroke (width 0) (type default) (color 0 0 0 0))
+  )
   (wire (pts (xy 102.362 80.518) (xy 106.172 80.518))
     (stroke (width 0) (type default) (color 0 0 0 0))
@@
     (stroke (width 0) (type default) (color 0 0 0 0))
   )
+  (wire (pts (xy 40.386 166.624) (xy 40.386 164.084))
+    (stroke (width 0) (type default) (color 0 0 0 0))
+  )
   (wire (pts (xy 102.616 28.448) (xy 106.426 28.448))
     (stroke (width 0) (type default) (color 0 0 0 0))
@@
     (stroke (width 0) (type default) (color 0 0 0 0))
   )
+  (wire (pts (xy 41.148 166.624) (xy 40.386 166.624))
+    (stroke (width 0) (type default) (color 0 0 0 0))
+  )
   (polyline (pts (xy 172.974 17.78) (xy 16.256 17.78))
     (stroke (width 0) (type default) (color 0 0 0 0))
@@
   )
   (wire (pts (xy 247.396 107.442) (xy 247.396 111.252))
+    (stroke (width 0) (type default) (color 0 0 0 0))
+  )
+  (wire (pts (xy 40.386 164.084) (xy 41.148 164.084))
     (stroke (width 0) (type default) (color 0 0 0 0))
   )
@@
   (text "Overvoltage Diode" (at 97.79 120.65 90)
     (effects (font (size 1.27 1.27)) (justify left bottom))
+  )
+  (global_label "Aux_In" (shape input) (at 129.794 176.53 180) (fields_autoplaced)
+    (effects (font (size 1.27 1.27)) (justify right))
+    (property "Intersheet References" "${INTERSHEET_REFS}" (id 0) (at 90.424 78.74 0)
+      (effects (font (size 1.27 1.27)) hide)
+    )
+  )
+  (global_label "BUCK_In" (shape output) (at 129.032 149.606 180) (fields_autoplaced)
+    (effects (font (size 1.27 1.27)) (justify right))
+    (property "Intersheet References" "${INTERSHEET_REFS}" (id 0) (at 118.8459 149.5266 0)
+      (effects (font (size 1.27 1.27)) (justify right) hide)
+    )
   )
   (global_label "V5" (shape output) (at 77.978 164.084 0) (fields_autoplaced)
@@
     )
   )
+  (global_label "VIN1" (shape input) (at 129.54 164.084 180) (fields_autoplaced)
+    (effects (font (size 1.27 1.27)) (justify right))
+    (property "Intersheet References" "${INTERSHEET_REFS}" (id 0) (at 122.9825 164.0046 0)
+      (effects (font (size 1.27 1.27)) (justify right) hide)
+    )
+  )
+  (global_label "Aux_In" (shape input) (at 129.54 159.004 180) (fields_autoplaced)
+    (effects (font (size 1.27 1.27)) (justify right))
+    (property "Intersheet References" "${INTERSHEET_REFS}" (id 0) (at 11.43 75.184 0)
+      (effects (font (size 1.27 1.27)) hide)
+    )
+  )
   (global_label "VIN1" (shape input) (at 69.596 28.956 90) (fields_autoplaced)
     (effects (font (size 1.27 1.27)) (justify left))
@@
     )
   )
-  (global_label "VIN1" (shape input) (at 33.528 164.084 180) (fields_autoplaced)
-    (effects (font (size 1.27 1.27)) (justify right))
-    (property "Intersheet References" "${INTERSHEET_REFS}" (id 0) (at 26.9705 164.0046 0)
+  (global_label "BUCK_In" (shape input) (at 33.528 164.084 180) (fields_autoplaced)
+    (effects (font (size 1.27 1.27)) (justify right))
+    (property "Intersheet References" "${INTERSHEET_REFS}" (id 0) (at 23.3419 164.0046 0)
       (effects (font (size 1.27 1.27)) (justify right) hide)
     )
@@
     )
   )
+  (global_label "V5" (shape output) (at 129.032 144.526 180) (fields_autoplaced)
+    (effects (font (size 1.27 1.27)) (justify right))
+    (property "Intersheet References" "${INTERSHEET_REFS}" (id 0) (at 124.4097 144.4466 0)
+      (effects (font (size 1.27 1.27)) (justify right) hide)
+    )
+  )
+  (global_label "Control_In" (shape output) (at 129.54 161.544 180) (fields_autoplaced)
+    (effects (font (size 1.27 1.27)) (justify right))
+    (property "Intersheet References" "${INTERSHEET_REFS}" (id 0) (at 117.6001 161.4646 0)
+      (effects (font (size 1.27 1.27)) (justify right) hide)
+    )
+  )
   (global_label "V2" (shape input) (at 20.32 64.77 180) (fields_autoplaced)
     (effects (font (size 1.27 1.27)) (justify right))
@@
     (effects (font (size 1.27 1.27)) (justify right))
     (property "Intersheet References" "${INTERSHEET_REFS}" (id 0) (at 251.1266 124.7643 90)
+      (effects (font (size 1.27 1.27)) (justify right) hide)
+    )
+  )
+  (global_label "Control_In" (shape input) (at 129.032 147.066 180) (fields_autoplaced)
+    (effects (font (size 1.27 1.27)) (justify right))
+    (property "Intersheet References" "${INTERSHEET_REFS}" (id 0) (at 117.0921 146.9866 0)
       (effects (font (size 1.27 1.27)) (justify right) hide)
     )
@@
     (pin "1")
   )
+  (symbol (lib_id "Connector_Generic:Conn_01x03") (at 134.112 147.066 0) (unit 1)
+    (in_bom yes) (on_board yes)
+    (property "Reference" "J34" (id 0) (at 136.144 145.9992 0)
+      (effects (font (size 1.27 1.27)) (justify left))
+    )
+    (property "Value" "Select Voltage" (id 1) (at 136.144 148.3106 0)
+      (effects (font (size 1.27 1.27)) (justify left))
+    )
+    (property "Footprint" "Connector_PinHeader_2.54mm:PinHeader_1x03_P2.54mm_Vertical" (id 2) (at 134.112 147.066 0)
+      (effects (font (size 1.27 1.27)) hide)
+    )
+    (property "Datasheet" "~" (id 3) (at 134.112 147.066 0)
+      (effects (font (size 1.27 1.27)) hide)
+    )
+    (pin "1")
+    (pin "2")
+    (pin "3")
+  )
   (symbol (lib_id "power:PWR_FLAG") (at 37.338 164.084 0) (unit 1)
     (in_bom yes) (on_board yes) (fields_autoplaced)
@@
       (effects (font (size 1.27 1.27)) hide)
     )
+    (pin "1")
+  )
+  (symbol (lib_id "Connector_Generic:Conn_01x03") (at 134.62 161.544 0) (unit 1)
+    (in_bom yes) (on_board yes)
+    (property "Reference" "J35" (id 0) (at 136.652 160.4772 0)
+      (effects (font (size 1.27 1.27)) (justify left))
+    )
+    (property "Value" "Select Control Feed" (id 1) (at 136.652 162.7886 0)
+      (effects (font (size 1.27 1.27)) (justify left))
+    )
+    (property "Footprint" "Connector_PinHeader_2.54mm:PinHeader_1x03_P2.54mm_Vertical" (id 2) (at 134.62 161.544 0)
+      (effects (font (size 1.27 1.27)) hide)
+    )
+    (property "Datasheet" "~" (id 3) (at 134.62 161.544 0)
+      (effects (font (size 1.27 1.27)) hide)
+    )
+    (pin "1")
+    (pin "2")
+    (pin "3")
+  )
+  (symbol (lib_id "Connector:Screw_Terminal_01x02") (at 134.874 179.07 0) (mirror x) (unit 1)
+    (in_bom yes) (on_board yes)
+    (property "Reference" "J36" (id 0) (at 136.906 178.8668 0)
+      (effects (font (size 1.27 1.27)) (justify left))
+    )
+    (property "Value" "Aux In" (id 1) (at 136.906 176.5554 0)
+      (effects (font (size 1.27 1.27)) (justify left))
+    )
+    (property "Footprint" "TerminalBlock_RND:TerminalBlock_RND_205-00012_1x02_P5.00mm_Horizontal" (id 2) (at 134.874 179.07 0)
+      (effects (font (size 1.27 1.27)) hide)
+    )
+    (property "Datasheet" "~" (id 3) (at 134.874 179.07 0)
+      (effects (font (size 1.27 1.27)) hide)
+    )
+    (pin "1")
+    (pin "2")
+  )
+  (symbol (lib_id "power:GND") (at 129.794 179.07 0) (unit 1)
+    (in_bom yes) (on_board yes)
+    (property "Reference" "#PWR0160" (id 0) (at 129.794 185.42 0)
+      (effects (font (size 1.27 1.27)) hide)
+    )
+    (property "Value" "GND" (id 1) (at 129.921 183.4642 0))
+    (property "Footprint" "" (id 2) (at 129.794 179.07 0)
+      (effects (font (size 1.27 1.27)) hide)
+    )
+    (property "Datasheet" "" (id 3) (at 129.794 179.07 0)
+      (effects (font (size 1.27 1.27)) hide)
+    )
