File: KiCAD/DPI-24/DPI-24-Controller/standard-hat-components.kicad_sch (KiCad schematic)
At the start: 12 parts, among them Q1 MMDT5401, Q2 DMG2302U, U1 AT24C256C

Commit message: addition of DPI-24 model
Parts:
- C2: value 0.1uF -> (none); footprint 3544again:C_0805_2012Metric -> (none)
- H1, H2, H3, H4: value M3 MountingHole -> (none); footprint MountingHole:MountingHole_3.2mm_M3_Pad_TopBottom -> (none)
- Q1: value MMDT5401 -> (none); footprint Package_TO_SOT_SMD:SOT-363_SC-70-6 -> (none)
- Q2: value DMG2302U -> (none); footprint Package_TO_SOT_SMD:SOT-23 -> (none)
- R25: renamed from R33; value 4.7k -> (none); footprint Resistor_SMD:R_0805_2012Metric -> (none)
- R27: renamed from R34; value 4.7k -> (none); footprint Resistor_SMD:R_0805_2012Metric -> (none)
- R35: value 10k -> (none); footprint Resistor_SMD:R_0805_2012Metric -> (none)
- R36: value 4.7k -> (none); footprint Resistor_SMD:R_0805_2012Metric -> (none)
- U1: value AT24C256C -> (none); footprint Package_SO:SOIC-8_3.9x4.9mm_P1.27mm -> (none)
Changed lines of the file:
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@@
       (effects (font (size 1.27 1.27)) (justify left))
     )
-    (property "Value" "M3 MountingHole" (id 1) (at 31.75 167.513 0)
-      (effects (font (size 1.27 1.27)) (justify left))
-    )
-    (property "Footprint" "MountingHole:MountingHole_3.2mm_M3_Pad_TopBottom" (id 2) (at 29.21 166.37 0)
+    (property "Value" "" (id 1) (at 31.75 167.513 0)
+      (effects (font (size 1.27 1.27)) (justify left))
+    )
+    (property "Footprint" "" (id 2) (at 29.21 166.37 0)
       (effects (font (size 1.27 1.27)) hide)
     )
@@
       (effects (font (size 1.27 1.27)) (justify left))
     )
-    (property "Value" "M3 MountingHole" (id 1) (at 31.75 172.593 0)
-      (effects (font (size 1.27 1.27)) (justify left))
-    )
-    (property "Footprint" "MountingHole:MountingHole_3.2mm_M3_Pad_TopBottom" (id 2) (at 29.21 171.45 0)
+    (property "Value" "" (id 1) (at 31.75 172.593 0)
+      (effects (font (size 1.27 1.27)) (justify left))
+    )
+    (property "Footprint" "" (id 2) (at 29.21 171.45 0)
       (effects (font (size 1.27 1.27)) hide)
     )
@@
       (effects (font (size 1.27 1.27)) (justify left))
     )
-    (property "Value" "M3 MountingHole" (id 1) (at 57.15 167.513 0)
-      (effects (font (size 1.27 1.27)) (justify left))
-    )
-    (property "Footprint" "MountingHole:MountingHole_3.2mm_M3_Pad_TopBottom" (id 2) (at 54.61 166.37 0)
+    (property "Value" "" (id 1) (at 57.15 167.513 0)
+      (effects (font (size 1.27 1.27)) (justify left))
+    )
+    (property "Footprint" "" (id 2) (at 54.61 166.37 0)
       (effects (font (size 1.27 1.27)) hide)
     )
@@
       (effects (font (size 1.27 1.27)) (justify left))
     )
-    (property "Value" "M3 MountingHole" (id 1) (at 57.15 172.593 0)
-      (effects (font (size 1.27 1.27)) (justify left))
-    )
-    (property "Footprint" "MountingHole:MountingHole_3.2mm_M3_Pad_TopBottom" (id 2) (at 54.61 171.45 0)
+    (property "Value" "" (id 1) (at 57.15 172.593 0)
+      (effects (font (size 1.27 1.27)) (justify left))
+    )
+    (property "Footprint" "" (id 2) (at 54.61 171.45 0)
       (effects (font (size 1.27 1.27)) hide)
     )
@@
       (effects (font (size 1.27 1.27)) (justify left))
     )
-    (property "Value" "4.7k" (id 1) (at 172.9486 78.613 0)
-      (effects (font (size 1.27 1.27)) (justify left))
-    )
-    (property "Footprint" "Resistor_SMD:R_0805_2012Metric" (id 2) (at 171.45 77.47 0)
+    (property "Value" "" (id 1) (at 172.9486 78.613 0)
+      (effects (font (size 1.27 1.27)) (justify left))
+    )
+    (property "Footprint" "" (id 2) (at 171.45 77.47 0)
       (effects (font (size 1.27 1.27)) hide)
     )
@@
   (symbol (lib_id "Device:R_Small") (at 66.04 74.93 0) (unit 1)
     (in_bom yes) (on_board yes)
-    (property "Reference" "R34" (id 0) (at 67.5386 73.7616 0)
-      (effects (font (size 1.27 1.27)) (justify left))
-    )
-    (property "Value" "4.7k" (id 1) (at 67.5386 76.073 0)
-      (effects (font (size 1.27 1.27)) (justify left))
-    )
-    (property "Footprint" "Resistor_SMD:R_0805_2012Metric" (id 2) (at 66.04 74.93 0)
+    (property "Reference" "R27" (id 0) (at 67.5386 73.7616 0)
+      (effects (font (size 1.27 1.27)) (justify left))
+    )
+    (property "Value" "" (id 1) (at 67.5386 76.073 0)
+      (effects (font (size 1.27 1.27)) (justify left))
+    )
+    (property "Footprint" "" (id 2) (at 66.04 74.93 0)
       (effects (font (size 1.27 1.27)) hide)
     )
@@
   (symbol (lib_id "Device:R_Small") (at 63.5 74.93 0) (unit 1)
     (in_bom yes) (on_board yes)
-    (property "Reference" "R33" (id 0) (at 64.9986 73.7616 90)
+    (property "Reference" "R25" (id 0) (at 64.9986 73.7616 90)
       (effects (font (size 1.27 1.27)) (justify left) hide)
     )
-    (property "Value" "4.7k" (id 1) (at 64.9986 76.073 0)
+    (property "Value" "" (id 1) (at 64.9986 76.073 0)
       (effects (font (size 1.27 1.27)) (justify left) hide)
     )
-    (property "Footprint" "Resistor_SMD:R_0805_2012Metric" (id 2) (at 63.5 74.93 0)
+    (property "Footprint" "" (id 2) (at 63.5 74.93 0)
       (effects (font (size 1.27 1.27)) hide)
     )
@@
     (in_bom yes) (on_board yes)
     (property "Reference" "U1" (id 0) (at 46.99 64.77 0))
-    (property "Value" "AT24C256C" (id 1) (at 46.99 67.31 0))
-    (property "Footprint" "Package_SO:SOIC-8_3.9x4.9mm_P1.27mm" (id 2) (at 48.26 85.09 0)
+    (property "Value" "" (id 1) (at 46.99 67.31 0))
+    (property "Footprint" "" (id 2) (at 48.26 85.09 0)
       (effects (font (size 1.27 1.27)) (justify bottom) hide)
     )
@@
       (effects (font (size 1.27 1.27)) (justify left))
     )
-    (property "Value" "10k" (id 1) (at 152.6286 78.613 0)
-      (effects (font (size 1.27 1.27)) (justify left))
-    )
-    (property "Footprint" "Resistor_SMD:R_0805_2012Metric" (id 2) (at 151.13 77.47 0)
+    (property "Value" "" (id 1) (at 152.6286 78.613 0)
+      (effects (font (size 1.27 1.27)) (justify left))
+    )
+    (property "Footprint" "" (id 2) (at 151.13 77.47 0)
       (effects (font (size 1.27 1.27)) hide)
     )
@@
     (in_bom yes) (on_board yes)
     (property "Reference" "Q2" (id 0) (at 161.29 42.1132 90))
-    (property "Value" "DMG2302U" (id 1) (at 161.29 44.4246 90))
-    (property "Footprint" "Package_TO_SOT_SMD:SOT-23" (id 2) (at 159.385 45.72 0)
+    (property "Value" "" (id 1) (at 161.29 44.4246 90))
+    (property "Footprint" "" (id 2) (at 159.385 45.72 0)
       (effects (font (size 1.27 1.27) italic) (justify left) hide)
     )
@@
       (effects (font (size 1.27 1.27)) (justify left))
     )
-    (property "Value" "MMDT5401" (id 1) (at 173.7614 62.357 0)
-      (effects (font (size 1.27 1.27)) (justify left))
-    )
-    (property "Footprint" "Package_TO_SOT_SMD:SOT-363_SC-70-6" (id 2) (at 173.99 66.04 0)
+    (property "Value" "" (id 1) (at 173.7614 62.357 0)
+      (effects (font (size 1.27 1.27)) (justify left))
+    )
+    (property "Footprint" "" (id 2) (at 173.99 66.04 0)
       (effects (font (size 1.27 1.27)) hide)
     )
@@
       (effects (font (size 1.27 1.27)) (justify left))
     )
-    (property "Value" "MMDT5401" (id 1) (at 148.8186 64.643 0)
-      (effects (font (size 1.27 1.27)) (justify left))
-    )
-    (property "Footprint" "Package_TO_SOT_SMD:SOT-363_SC-70-6" (id 2) (at 148.59 66.04 0)
+    (property "Value" "" (id 1) (at 148.8186 64.643 0)
+      (effects (font (size 1.27 1.27)) (justify left))
+    )
+    (property "Footprint" "" (id 2) (at 148.59 66.04 0)
       (effects (font (size 1.27 1.27)) hide)
     )
@@
     (in_bom yes) (on_board yes)
     (property "Reference" "C2" (id 0) (at 40.64 69.1134 90))
-    (property "Value" "0.1uF" (id 1) (at 40.64 71.4248 90))
-    (property "Footprint" "3544again:C_0805_2012Metric" (id 2) (at 40.64 74.93 0)
-      (effects (font (size 1.27 1.27)) hide)
-    )
+    (property "Value" "" (id 1) (at 40.64 71.4248 90))
+    (property "Footprint" "" (id 2) (at 40.64 74.93 0)
+      (effects (font (size 1.27 1.27)) hide)
+    )

Commit message: layout updates
Parts:
- C2: value (none) -> 0.1uF; footprint (none) -> Capacitor_THT:C_Radial_D5.0mm_H11.0mm_P2.00mm
- H1, H2, H3, H4: value (none) -> M3 MountingHole; footprint (none) -> MountingHole:MountingHole_3.2mm_M3_Pad_TopBottom
- Q1: value (none) -> MMDT5401; footprint (none) -> Package_TO_SOT_SMD:SOT-363_SC-70-6
- Q2: value (none) -> DMG2302U; footprint (none) -> Package_TO_SOT_SMD:SOT-23
- R25, R27, R36: value (none) -> 4.7k; footprint (none) -> Resistor_SMD:R_0805_2012Metric
- R35: value (none) -> 10k; footprint (none) -> Resistor_SMD:R_0805_2012Metric
- U1: value (none) -> AT24C256C; footprint (none) -> Package_DIP:DIP-8_W7.62mm_Socket
Other:
- title: The Owl - RPI Cape 16ch Pixel Controller -> RPI Cape DPI 24ch Pixel Controller
Changed lines of the file:
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@@
   (paper "A4")
   (title_block
-    (title "The Owl - RPI Cape 16ch Pixel Controller")
+    (title "RPI Cape DPI 24ch Pixel Controller")
     (date "2022-04-04")
     (company "OnlineDynamic")
@@
       (effects (font (size 1.27 1.27)) (justify left))
     )
-    (property "Value" "" (id 1) (at 31.75 167.513 0)
-      (effects (font (size 1.27 1.27)) (justify left))
-    )
-    (property "Footprint" "" (id 2) (at 29.21 166.37 0)
+    (property "Value" "M3 MountingHole" (id 1) (at 31.75 167.513 0)
+      (effects (font (size 1.27 1.27)) (justify left))
+    )
+    (property "Footprint" "MountingHole:MountingHole_3.2mm_M3_Pad_TopBottom" (id 2) (at 29.21 166.37 0)
       (effects (font (size 1.27 1.27)) hide)
     )
@@
       (effects (font (size 1.27 1.27)) (justify left))
     )
-    (property "Value" "" (id 1) (at 31.75 172.593 0)
-      (effects (font (size 1.27 1.27)) (justify left))
-    )
-    (property "Footprint" "" (id 2) (at 29.21 171.45 0)
+    (property "Value" "M3 MountingHole" (id 1) (at 31.75 172.593 0)
+      (effects (font (size 1.27 1.27)) (justify left))
+    )
+    (property "Footprint" "MountingHole:MountingHole_3.2mm_M3_Pad_TopBottom" (id 2) (at 29.21 171.45 0)
       (effects (font (size 1.27 1.27)) hide)
     )
@@
       (effects (font (size 1.27 1.27)) (justify left))
     )
-    (property "Value" "" (id 1) (at 57.15 167.513 0)
-      (effects (font (size 1.27 1.27)) (justify left))
-    )
-    (property "Footprint" "" (id 2) (at 54.61 166.37 0)
+    (property "Value" "M3 MountingHole" (id 1) (at 57.15 167.513 0)
+      (effects (font (size 1.27 1.27)) (justify left))
+    )
+    (property "Footprint" "MountingHole:MountingHole_3.2mm_M3_Pad_TopBottom" (id 2) (at 54.61 166.37 0)
       (effects (font (size 1.27 1.27)) hide)
     )
@@
       (effects (font (size 1.27 1.27)) (justify left))
     )
-    (property "Value" "" (id 1) (at 57.15 172.593 0)
-      (effects (font (size 1.27 1.27)) (justify left))
-    )
-    (property "Footprint" "" (id 2) (at 54.61 171.45 0)
+    (property "Value" "M3 MountingHole" (id 1) (at 57.15 172.593 0)
+      (effects (font (size 1.27 1.27)) (justify left))
+    )
+    (property "Footprint" "MountingHole:MountingHole_3.2mm_M3_Pad_TopBottom" (id 2) (at 54.61 171.45 0)
       (effects (font (size 1.27 1.27)) hide)
     )
@@
       (effects (font (size 1.27 1.27)) (justify left))
     )
-    (property "Value" "" (id 1) (at 172.9486 78.613 0)
-      (effects (font (size 1.27 1.27)) (justify left))
-    )
-    (property "Footprint" "" (id 2) (at 171.45 77.47 0)
+    (property "Value" "4.7k" (id 1) (at 172.9486 78.613 0)
+      (effects (font (size 1.27 1.27)) (justify left))
+    )
+    (property "Footprint" "Resistor_SMD:R_0805_2012Metric" (id 2) (at 171.45 77.47 0)
       (effects (font (size 1.27 1.27)) hide)
     )
@@
       (effects (font (size 1.27 1.27)) (justify left))
     )
-    (property "Value" "" (id 1) (at 67.5386 76.073 0)
-      (effects (font (size 1.27 1.27)) (justify left))
-    )
-    (property "Footprint" "" (id 2) (at 66.04 74.93 0)
+    (property "Value" "4.7k" (id 1) (at 67.5386 76.073 0)
+      (effects (font (size 1.27 1.27)) (justify left))
+    )
+    (property "Footprint" "Resistor_SMD:R_0805_2012Metric" (id 2) (at 66.04 74.93 0)
       (effects (font (size 1.27 1.27)) hide)
     )
@@
       (effects (font (size 1.27 1.27)) (justify left) hide)
     )
-    (property "Value" "" (id 1) (at 64.9986 76.073 0)
+    (property "Value" "4.7k" (id 1) (at 64.9986 76.073 0)
       (effects (font (size 1.27 1.27)) (justify left) hide)
     )
-    (property "Footprint" "" (id 2) (at 63.5 74.93 0)
+    (property "Footprint" "Resistor_SMD:R_0805_2012Metric" (id 2) (at 63.5 74.93 0)
       (effects (font (size 1.27 1.27)) hide)
     )
@@
     (in_bom yes) (on_board yes)
     (property "Reference" "U1" (id 0) (at 46.99 64.77 0))
-    (property "Value" "" (id 1) (at 46.99 67.31 0))
-    (property "Footprint" "" (id 2) (at 48.26 85.09 0)
+    (property "Value" "AT24C256C" (id 1) (at 46.99 67.31 0))
+    (property "Footprint" "Package_DIP:DIP-8_W7.62mm_Socket" (id 2) (at 48.26 85.09 0)
       (effects (font (size 1.27 1.27)) (justify bottom) hide)
     )
@@
       (effects (font (size 1.27 1.27)) (justify left))
     )
-    (property "Value" "" (id 1) (at 152.6286 78.613 0)
-      (effects (font (size 1.27 1.27)) (justify left))
-    )
-    (property "Footprint" "" (id 2) (at 151.13 77.47 0)
+    (property "Value" "10k" (id 1) (at 152.6286 78.613 0)
+      (effects (font (size 1.27 1.27)) (justify left))
+    )
+    (property "Footprint" "Resistor_SMD:R_0805_2012Metric" (id 2) (at 151.13 77.47 0)
       (effects (font (size 1.27 1.27)) hide)
     )
@@
     (in_bom yes) (on_board yes)
     (property "Reference" "Q2" (id 0) (at 161.29 42.1132 90))
-    (property "Value" "" (id 1) (at 161.29 44.4246 90))
-    (property "Footprint" "" (id 2) (at 159.385 45.72 0)
+    (property "Value" "DMG2302U" (id 1) (at 161.29 44.4246 90))
+    (property "Footprint" "Package_TO_SOT_SMD:SOT-23" (id 2) (at 159.385 45.72 0)
       (effects (font (size 1.27 1.27) italic) (justify left) hide)
     )
@@
       (effects (font (size 1.27 1.27)) (justify left))
     )
-    (property "Value" "" (id 1) (at 173.7614 62.357 0)
-      (effects (font (size 1.27 1.27)) (justify left))
-    )
-    (property "Footprint" "" (id 2) (at 173.99 66.04 0)
+    (property "Value" "MMDT5401" (id 1) (at 173.7614 62.357 0)
+      (effects (font (size 1.27 1.27)) (justify left))
+    )
+    (property "Footprint" "Package_TO_SOT_SMD:SOT-363_SC-70-6" (id 2) (at 173.99 66.04 0)
       (effects (font (size 1.27 1.27)) hide)
     )
@@
       (effects (font (size 1.27 1.27)) (justify left))
     )
-    (property "Value" "" (id 1) (at 148.8186 64.643 0)
-      (effects (font (size 1.27 1.27)) (justify left))
-    )
-    (property "Footprint" "" (id 2) (at 148.59 66.04 0)
+    (property "Value" "MMDT5401" (id 1) (at 148.8186 64.643 0)
+      (effects (font (size 1.27 1.27)) (justify left))
+    )
+    (property "Footprint" "Package_TO_SOT_SMD:SOT-363_SC-70-6" (id 2) (at 148.59 66.04 0)
       (effects (font (size 1.27 1.27)) hide)
     )
@@
     (in_bom yes) (on_board yes)
     (property "Reference" "C2" (id 0) (at 40.64 69.1134 90))
-    (property "Value" "" (id 1) (at 40.64 71.4248 90))
-    (property "Footprint" "" (id 2) (at 40.64 74.93 0)
-      (effects (font (size 1.27 1.27)) hide)
-    )
-    (property "Datasheet" "https://datasheet.lcsc.com/szlcsc/Samsung-Electro-Mechanics-CL05B104KO5NNNC_C1525.pdf" (id 3) (at 40.64 74.93 0)
-      (effects (font (size 1.27 1.27)) hide)
-    )
-    (property "Description" "C49678" (id 4) (at 40.64 74.93 0)
-      (effects (font (size 1.27 1.27)) hide)
-    )
+    (property "Value" "0.1uF" (id 1) (at 40.64 71.4248 90))
+    (property "Footprint" "Capacitor_THT:C_Radial_D5.0mm_H11.0mm_P2.00mm" (id 2) (at 40.64 74.93 0)
+      (effects (font (size 1.27 1.27)) hide)
+    )
+    (property "Datasheet" "" (id 3) (at 40.64 74.93 0)
+      (effects (font (size 1.27 1.27)) hide)
+    )
+    (property "Description" "" (id 4) (at 40.64 74.93 0)
+      (effects (font (size 1.27 1.27)) hide)
+    )
