File: KiCAD/DPI-24/DPI-24-Controller/_autosave-controls.kicad_sch (KiCad schematic)
At the start: 14 parts, among them J32 OLED, J33 GPIO TRG, SW1 SW_UP, SW2 SW_DOWN, SW3 SW_BACK, SW4 SW_TEST, SW5 SW_ENTER, U3 TZT_Original_0.96_inch_oled_I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

Commit message: further layout updates
Parts:
- SW1: value SW_UP -> UP
- SW2: value SW_DOWN -> DOWN
- SW3: value SW_BACK -> BACK
- SW4: value SW_TEST -> TEST
- SW5: value SW_ENTER -> ENTER
Changed lines of the file:
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@@
     (in_bom yes) (on_board yes) (fields_autoplaced)
     (property "Reference" "SW4" (id 0) (at 42.672 126.7292 0))
-    (property "Value" "SW_TEST" (id 1) (at 42.672 129.2661 0))
+    (property "Value" "TEST" (id 1) (at 42.672 129.2661 0))
     (property "Footprint" "Button_Switch_THT:SW_PUSH_6mm" (id 2) (at 42.672 128.27 0)
       (effects (font (size 1.27 1.27)) hide)
@@
     (in_bom yes) (on_board yes) (fields_autoplaced)
     (property "Reference" "SW1" (id 0) (at 42.672 91.1692 0))
-    (property "Value" "SW_UP" (id 1) (at 42.672 93.7061 0))
+    (property "Value" "UP" (id 1) (at 42.672 93.7061 0))
     (property "Footprint" "Button_Switch_THT:SW_PUSH_6mm" (id 2) (at 42.672 92.71 0)
       (effects (font (size 1.27 1.27)) hide)
@@
     (in_bom yes) (on_board yes) (fields_autoplaced)
     (property "Reference" "SW3" (id 0) (at 42.672 114.0292 0))
-    (property "Value" "SW_BACK" (id 1) (at 42.672 116.5661 0))
+    (property "Value" "BACK" (id 1) (at 42.672 116.5661 0))
     (property "Footprint" "Button_Switch_THT:SW_PUSH_6mm" (id 2) (at 42.672 115.57 0)
       (effects (font (size 1.27 1.27)) hide)
@@
     (in_bom yes) (on_board yes) (fields_autoplaced)
     (property "Reference" "SW2" (id 0) (at 42.672 102.5992 0))
-    (property "Value" "SW_DOWN" (id 1) (at 42.672 105.1361 0))
+    (property "Value" "DOWN" (id 1) (at 42.672 105.1361 0))
     (property "Footprint" "Button_Switch_THT:SW_PUSH_6mm" (id 2) (at 42.672 104.14 0)
       (effects (font (size 1.27 1.27)) hide)
@@
     (in_bom yes) (on_board yes) (fields_autoplaced)
     (property "Reference" "SW5" (id 0) (at 42.672 139.4292 0))
-    (property "Value" "SW_ENTER" (id 1) (at 42.672 141.9661 0))
+    (property "Value" "ENTER" (id 1) (at 42.672 141.9661 0))
     (property "Footprint" "Button_Switch_THT:SW_PUSH_6mm" (id 2) (at 42.672 140.97 0)
       (effects (font (size 1.27 1.27)) hide)
