File: KiCAD/DPI-24/DPI-24-Controller/_autosave-power.kicad_sch (KiCad schematic)
At the start: 20 parts, among them J28 1-8 In, J29 9-16 In 12V DC, J30 17-24 In 12V DC, U2 D-SUN_MP1584_BUCK

Commit message: further layout updates
Parts:
- J28: value 1-8 In -> Ports 1-8 12V DC IN
- J29: value 9-16 In 12V DC -> Ports 9-16 12V DC IN
- J30: value 17-24 In 12V DC -> Ports 17-24 12V DC IN
Changed lines of the file:
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@@
       (effects (font (size 1.27 1.27)) (justify left))
     )
-    (property "Value" "1-8 In" (id 1) (at 54.102 29.2354 0)
+    (property "Value" "Ports 1-8 12V DC IN" (id 1) (at 54.102 29.2354 0)
       (effects (font (size 1.27 1.27)) (justify left))
     )
@@
       (effects (font (size 1.27 1.27)) (justify left))
     )
-    (property "Value" "9-16 In 12V DC" (id 1) (at 50.292 64.7954 0)
+    (property "Value" "Ports 9-16 12V DC IN" (id 1) (at 50.292 64.7954 0)
       (effects (font (size 1.27 1.27)) (justify left))
     )
@@
       (effects (font (size 1.27 1.27)) (justify left))
     )
-    (property "Value" "17-24 In 12V DC" (id 1) (at 195.326 104.4194 0)
-      (effects (font (size 1.27 1.27)) (justify left))
-    )
+    (property "Value" "Ports 17-24 12V DC IN" (id 1) (at 184.658 101.6 0)
+      (effects (font (size 1.27 1.27)) (justify left))
+    )
