File: KiCAD/DPI-24/DPI-24-Controller/ethernet.kicad_sch (KiCad schematic)
At the start: 11 parts

Commit message: layout updates
Parts:
- D33, D34: value (none) -> 0603; footprint (none) -> LED_SMD:LED_0603_1608Metric
- IC5: value (none) -> KSZ8794CNXIC; footprint (none) -> QFN40P800X800X90-65N
- J25: value (none) -> UPLINK; footprint (none) -> Connector_RJ:RJ45_BEL_SS74301-00x_Vertical
- J26: value (none) -> LAN 1; footprint (none) -> Connector_RJ:RJ45_BEL_SS74301-00x_Vertical
- J27: value (none) -> LAN 2; footprint (none) -> Connector_RJ:RJ45_BEL_SS74301-00x_Vertical
- R28, R29: value (none) -> 4.7k; footprint (none) -> Resistor_SMD:R_0805_2012Metric
- R46: value (none) -> 12k; footprint (none) -> Resistor_SMD:R_0805_2012Metric
- R47: value (none) -> 8.06K; footprint (none) -> Resistor_SMD:R_0805_2012Metric
- U4: value (none) -> LAN7500-ABJZ; footprint (none) -> Package_DFN_QFN:QFN-56-1EP_8x8mm_P0.5mm_EP5.9x5.9mm
Other:
- title: The Owl - RPI Cape 16ch Pixel Controller -> RPI Cape DPI 24ch Pixel Controller
Changed lines of the file:
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@@
   (paper "A4")
   (title_block
-    (title "The Owl - RPI Cape 16ch Pixel Controller")
+    (title "RPI Cape DPI 24ch Pixel Controller")
     (date "2022-04-04")
     (company "OnlineDynamic")
@@
       (effects (font (size 1.27 1.27)) (justify left))
     )
-    (property "Value" "" (id 1) (at 262.636 35.4842 90)
-      (effects (font (size 1.27 1.27)) (justify left))
-    )
-    (property "Footprint" "" (id 2) (at 249.809 33.782 90)
+    (property "Value" "UPLINK" (id 1) (at 262.636 35.4842 90)
+      (effects (font (size 1.27 1.27)) (justify left))
+    )
+    (property "Footprint" "Connector_RJ:RJ45_BEL_SS74301-00x_Vertical" (id 2) (at 249.809 33.782 90)
       (effects (font (size 1.27 1.27)) hide)
     )
@@
     (in_bom yes) (on_board yes) (fields_autoplaced)
     (property "Reference" "IC5" (id 0) (at 249.1965 84.4635 0))
-    (property "Value" "" (id 1) (at 249.1965 87.0004 0))
-    (property "Footprint" "" (id 2) (at 242.57 69.85 0)
+    (property "Value" "KSZ8794CNXIC" (id 1) (at 249.1965 87.0004 0))
+    (property "Footprint" "QFN40P800X800X90-65N" (id 2) (at 242.57 69.85 0)
       (effects (font (size 1.27 1.27)) (justify left) hide)
     )
@@
       (effects (font (size 1.27 1.27)) hide)
     )
-    (property "Value" "" (id 1) (at 249.555 116.0038 90)
+    (property "Value" "GND" (id 1) (at 249.555 116.0038 90)
       (effects (font (size 1.27 1.27)) (justify right))
     )
@@
       (effects (font (size 1.27 1.27)) hide)
     )
-    (property "Value" "" (id 1) (at 198.12 153.0334 0))
+    (property "Value" "GND" (id 1) (at 198.12 153.0334 0))
     (property "Footprint" "" (id 2) (at 198.12 148.59 0)
       (effects (font (size 1.27 1.27)) hide)
@@
       (effects (font (size 1.27 1.27)) hide)
     )
-    (property "Value" "" (id 1) (at 216.154 19.2842 0))
+    (property "Value" "GND" (id 1) (at 216.154 19.2842 0))
     (property "Footprint" "" (id 2) (at 216.154 22.86 0)
       (effects (font (size 1.27 1.27)) hide)
@@
       (effects (font (size 1.27 1.27)) (justify left))
     )
-    (property "Value" "" (id 1) (at 187.706 34.7222 90)
-      (effects (font (size 1.27 1.27)) (justify left))
-    )
-    (property "Footprint" "" (id 2) (at 174.879 33.02 90)
+    (property "Value" "LAN 1" (id 1) (at 187.706 34.7222 90)
+      (effects (font (size 1.27 1.27)) (justify left))
+    )
+    (property "Footprint" "Connector_RJ:RJ45_BEL_SS74301-00x_Vertical" (id 2) (at 174.879 33.02 90)
       (effects (font (size 1.27 1.27)) hide)
     )
@@
       (effects (font (size 1.27 1.27)) (justify right))
     )
-    (property "Value" "" (id 1) (at 132.334 118.872 90)
+    (property "Value" "0603" (id 1) (at 132.334 118.872 90)
       (effects (font (size 1.27 1.27)) (justify right))
     )
-    (property "Footprint" "" (id 2) (at 129.794 116.332 0)
+    (property "Footprint" "LED_SMD:LED_0603_1608Metric" (id 2) (at 129.794 116.332 0)
       (effects (font (size 1.27 1.27)) hide)
     )
@@
       (effects (font (size 1.27 1.27)) (justify left))
     )
-    (property "Value" "" (id 1) (at 70.5994 145.5373 0)
-      (effects (font (size 1.27 1.27)) (justify left))
-    )
-    (property "Footprint" "" (id 2) (at 100.33 142.24 0)
+    (property "Value" "LAN7500-ABJZ" (id 1) (at 70.5994 145.5373 0)
+      (effects (font (size 1.27 1.27)) (justify left))
+    )
+    (property "Footprint" "Package_DFN_QFN:QFN-56-1EP_8x8mm_P0.5mm_EP5.9x5.9mm" (id 2) (at 100.33 142.24 0)
       (effects (font (size 1.27 1.27)) hide)
     )
@@
       (effects (font (size 1.27 1.27)) (justify right))
     )
-    (property "Value" "" (id 1) (at 143.002 114.3 90)
+    (property "Value" "0603" (id 1) (at 143.002 114.3 90)
       (effects (font (size 1.27 1.27)) (justify right))
     )
-    (property "Footprint" "" (id 2) (at 140.462 111.76 0)
+    (property "Footprint" "LED_SMD:LED_0603_1608Metric" (id 2) (at 140.462 111.76 0)
       (effects (font (size 1.27 1.27)) hide)
     )
@@
       (effects (font (size 1.27 1.27)) (justify left))
     )
-    (property "Value" "" (id 1) (at 219.456 34.7222 90)
-      (effects (font (size 1.27 1.27)) (justify left))
-    )
-    (property "Footprint" "" (id 2) (at 206.629 33.02 90)
+    (property "Value" "LAN 2" (id 1) (at 219.456 34.7222 90)
+      (effects (font (size 1.27 1.27)) (justify left))
+    )
+    (property "Footprint" "Connector_RJ:RJ45_BEL_SS74301-00x_Vertical" (id 2) (at 206.629 33.02 90)
       (effects (font (size 1.27 1.27)) hide)
     )
@@
       (effects (font (size 1.27 1.27)) (justify left))
     )
-    (property "Value" "" (id 1) (at 41.783 50.5714 0)
-      (effects (font (size 1.27 1.27)) (justify left))
-    )
-    (property "Footprint" "" (id 2) (at 40.64 52.07 0)
+    (property "Value" "12k" (id 1) (at 41.783 50.5714 0)
+      (effects (font (size 1.27 1.27)) (justify left))
+    )
+    (property "Footprint" "Resistor_SMD:R_0805_2012Metric" (id 2) (at 40.64 52.07 0)
       (effects (font (size 1.27 1.27)) hide)
     )
@@
       (effects (font (size 1.27 1.27)) (justify left))
     )
-    (property "Value" "" (id 1) (at 41.783 56.9214 0)
-      (effects (font (size 1.27 1.27)) (justify left))
-    )
-    (property "Footprint" "" (id 2) (at 40.64 58.42 0)
+    (property "Value" "8.06K" (id 1) (at 41.783 56.9214 0)
+      (effects (font (size 1.27 1.27)) (justify left))
+    )
+    (property "Footprint" "Resistor_SMD:R_0805_2012Metric" (id 2) (at 40.64 58.42 0)
       (effects (font (size 1.27 1.27)) hide)
     )
@@
     (in_bom yes) (on_board yes) (fields_autoplaced)
     (property "Reference" "U4" (id 0) (at 63.5 30.5902 0))
-    (property "Value" "" (id 1) (at 63.5 33.1271 0))
-    (property "Footprint" "" (id 2) (at 95.25 78.74 0)
+    (property "Value" "LAN7500-ABJZ" (id 1) (at 63.5 33.1271 0))
+    (property "Footprint" "Package_DFN_QFN:QFN-56-1EP_8x8mm_P0.5mm_EP5.9x5.9mm" (id 2) (at 95.25 78.74 0)
       (effects (font (size 1.27 1.27)) hide)
     )
@@
       (effects (font (size 1.27 1.27)) (justify left))
     )
-    (property "Value" "" (id 1) (at 131.2926 111.125 0)
-      (effects (font (size 1.27 1.27)) (justify left))
-    )
-    (property "Footprint" "" (id 2) (at 129.794 109.982 0)
+    (property "Value" "4.7k" (id 1) (at 131.2926 111.125 0)
+      (effects (font (size 1.27 1.27)) (justify left))
+    )
+    (property "Footprint" "Resistor_SMD:R_0805_2012Metric" (id 2) (at 129.794 109.982 0)
       (effects (font (size 1.27 1.27)) hide)
     )
@@
       (effects (font (size 1.27 1.27)) (justify left))
     )
-    (property "Value" "" (id 1) (at 141.9606 106.553 0)
-      (effects (font (size 1.27 1.27)) (justify left))
-    )
-    (property "Footprint" "" (id 2) (at 140.462 105.41 0)
-      (effects (font (size 1.27 1.27)) hide)
-    )
+    (property "Value" "4.7k" (id 1) (at 141.9606 106.553 0)
+      (effects (font (size 1.27 1.27)) (justify left))
+    )
+    (property "Footprint" "Resistor_SMD:R_0805_2012Metric" (id 2) (at 140.462 105.41 0)
+      (effects (font (size 1.27 1.27)) hide)
+    )

Commit message: further layout updates
Parts:
- IC5: footprint QFN40P800X800X90-65N -> SamacSys_Parts:QFN40P800X800X90-65N
Changed lines of the file:
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@@
     (property "Reference" "IC5" (id 0) (at 249.1965 84.4635 0))
     (property "Value" "KSZ8794CNXIC" (id 1) (at 249.1965 87.0004 0))
-    (property "Footprint" "QFN40P800X800X90-65N" (id 2) (at 242.57 69.85 0)
+    (property "Footprint" "SamacSys_Parts:QFN40P800X800X90-65N" (id 2) (at 242.57 69.85 0)
       (effects (font (size 1.27 1.27)) (justify left) hide)
     )
