File: KiCAD/DPI-24/DPI-24-Controller/out-ports1-8.kicad_sch (KiCad schematic)
At the start: 36 parts

Commit message: layout updates
Parts:
- C1: value (none) -> 0.1uF; footprint (none) -> Capacitor_THT:C_Radial_D5.0mm_H11.0mm_P2.00mm
- D1, D2, D3, D4, D5, D6, D7, D8: value (none) -> 0603; footprint (none) -> LED_SMD:LED_0603_1608Metric
- F1: value (none) -> P1; footprint (none) -> Stuart_BESPOKE:Medium Auto Fuse Holder
- F2: value (none) -> P2; footprint (none) -> Stuart_BESPOKE:Medium Auto Fuse Holder
- F3: value (none) -> P3; footprint (none) -> Stuart_BESPOKE:Medium Auto Fuse Holder
- F4: value (none) -> P4; footprint (none) -> Stuart_BESPOKE:Medium Auto Fuse Holder
- F5: value (none) -> P5; footprint (none) -> Stuart_BESPOKE:Medium Auto Fuse Holder
- F6: value (none) -> P6; footprint (none) -> Stuart_BESPOKE:Medium Auto Fuse Holder
- F7: value (none) -> P7; footprint (none) -> Stuart_BESPOKE:Medium Auto Fuse Holder
- F8: value (none) -> P8; footprint (none) -> Stuart_BESPOKE:Medium Auto Fuse Holder
- IC1: value (none) -> SN74AHC245N; footprint (none) -> DIP794W53P254L2540H508Q20N
- J1, J2, J3, J4, J5, J6, J7, J8: value (none) -> G D V; footprint (none) -> Connector_Phoenix_MC:PhoenixContact_MCV_1,5_3-G-3.5_1x03_P3.50mm_Vertical
- R1, R2, R3, R4, R5, R6, R7, R8: value (none) -> 4.7k; footprint (none) -> Resistor_SMD:R_0805_2012Metric
- RN1, RN2: value (none) -> 33R; footprint (none) -> Resistor_THT:R_Array_SIP8
Other:
- title: The Owl - RPI Cape 16ch Pixel Controller -> RPI Cape DPI 24ch Pixel Controller

Commit message: further layout updates
Parts:
- IC1: footprint DIP794W53P254L2540H508Q20N -> SamacSys_Parts:DIP794W53P254L2540H508Q20N
Changed lines of the file:
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@@
     (property "Reference" "IC1" (id 0) (at 43.18 94.141 0))
     (property "Value" "SN74AHC245N" (id 1) (at 43.18 96.6779 0))
-    (property "Footprint" "DIP794W53P254L2540H508Q20N" (id 2) (at 52.07 97.79 0)
+    (property "Footprint" "SamacSys_Parts:DIP794W53P254L2540H508Q20N" (id 2) (at 52.07 97.79 0)
       (effects (font (size 1.27 1.27)) (justify left) hide)
     )
