File: KiCAD/DPI-24/DPI-24-Controller/outports9-16.kicad_sch (KiCad schematic)
At the start: 36 parts

Commit message: layout updates
Parts:
- C3: value (none) -> 0.1uF; footprint (none) -> Capacitor_THT:C_Radial_D5.0mm_H11.0mm_P2.00mm
- D10, D11, D12, D13, D14, D15, D16, D9: value (none) -> 0603; footprint (none) -> LED_SMD:LED_0603_1608Metric
- F10, F11, F12, F13, F14, F15, F16, F9: value (none) -> P1; footprint (none) -> Stuart_BESPOKE:Medium Auto Fuse Holder
- IC2: value (none) -> SN74AHC245N; footprint (none) -> DIP794W53P254L2540H508Q20N
- J10, J11, J12, J13, J14, J15, J16, J9: value (none) -> G D V; footprint (none) -> Connector_Phoenix_MC:PhoenixContact_MCV_1,5_3-G-3.5_1x03_P3.50mm_Vertical
- R10, R11, R12, R13, R14, R15, R16, R9: value (none) -> 4.7k; footprint (none) -> Resistor_SMD:R_0805_2012Metric
- RN3, RN4: value (none) -> 33R; footprint (none) -> Resistor_THT:R_Array_SIP8
Other:
- title: The Owl - RPI Cape 16ch Pixel Controller -> RPI Cape DPI 24ch Pixel Controller

Commit message: further layout updates
Parts:
- IC2: footprint DIP794W53P254L2540H508Q20N -> SamacSys_Parts:DIP794W53P254L2540H508Q20N
Changed lines of the file:
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@@
     (property "Reference" "IC2" (id 0) (at 41.91 94.141 0))
     (property "Value" "SN74AHC245N" (id 1) (at 41.91 96.6779 0))
-    (property "Footprint" "DIP794W53P254L2540H508Q20N" (id 2) (at 50.8 97.79 0)
+    (property "Footprint" "SamacSys_Parts:DIP794W53P254L2540H508Q20N" (id 2) (at 50.8 97.79 0)
       (effects (font (size 1.27 1.27)) (justify left) hide)
     )
