File: KiCAD/DPI-24/DPI-24-Controller/DPI-24-Controller.kicad_sch (KiCad schematic)
At the start: 2 parts

Commit message: dpi-24 updates
Parts:
- added H5, H6: (no value), symbol Mechanical:MountingHole_Pad
Connections:
- net USBDM: now also H5.1
- net USBDP: now also H6.1
Changed lines of the file:
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@@
+    (stroke (width 0) (type default) (color 0 0 0 0))
+  )
+  (wire (pts (xy 30.734 185.674) (xy 40.894 185.674))
     (stroke (width 0) (type default) (color 0 0 0 0))
   )
@@
     (stroke (width 0) (type default) (color 0 0 0 0))
   )
+  (wire (pts (xy 40.894 185.674) (xy 40.894 181.864))
+    (stroke (width 0) (type default) (color 0 0 0 0))
+  )
   (wire (pts (xy 37.592 40.64) (xy 40.64 40.64))
     (stroke (width 0) (type default) (color 0 0 0 0))
@@
     (stroke (width 0) (type default) (color 0 0 0 0))
   )
+  (wire (pts (xy 45.974 181.864) (xy 45.974 185.674))
+    (stroke (width 0) (type default) (color 0 0 0 0))
+  )
   (wire (pts (xy 36.83 55.88) (xy 40.64 55.88))
     (stroke (width 0) (type default) (color 0 0 0 0))
@@
   )
   (wire (pts (xy 36.83 63.5) (xy 40.64 63.5))
+    (stroke (width 0) (type default) (color 0 0 0 0))
+  )
+  (wire (pts (xy 56.896 185.674) (xy 45.974 185.674))
     (stroke (width 0) (type default) (color 0 0 0 0))
   )
@@
     )
   )
+  (global_label "USBDM" (shape bidirectional) (at 40.894 181.864 90) (fields_autoplaced)
+    (effects (font (size 1.27 1.27)) (justify left))
+    (property "Intersheet References" "${INTERSHEET_REFS}" (id 0) (at 40.8146 173.0084 90)
+      (effects (font (size 1.27 1.27)) (justify left) hide)
+    )
+  )
   (global_label "I2C_SCL" (shape bidirectional) (at 37.592 43.18 180) (fields_autoplaced)
     (effects (font (size 1.27 1.27)) (justify right))
@@
     (property "Intersheet References" "${INTERSHEET_REFS}" (id 0) (at 28.8815 76.1206 0)
       (effects (font (size 1.27 1.27)) (justify right) hide)
+    )
+  )
+  (global_label "USBDP" (shape bidirectional) (at 45.974 181.864 90) (fields_autoplaced)
+    (effects (font (size 1.27 1.27)) (justify left))
+    (property "Intersheet References" "${INTERSHEET_REFS}" (id 0) (at 46.0534 173.1898 90)
+      (effects (font (size 1.27 1.27)) (justify left) hide)
     )
   )
@@
     )
     (property "Datasheet" "" (id 3) (at 53.34 40.64 0)
+      (effects (font (size 1.27 1.27)) hide)
+    )
+    (pin "1")
+  )
+  (symbol (lib_id "Mechanical:MountingHole_Pad") (at 56.896 188.214 180) (unit 1)
+    (in_bom yes) (on_board yes) (fields_autoplaced)
+    (property "Reference" "H6" (id 0) (at 59.436 188.6493 0)
+      (effects (font (size 1.27 1.27)) (justify right))
+    )
+    (property "Value" "" (id 1) (at 59.436 191.1862 0)
+      (effects (font (size 1.27 1.27)) (justify right))
+    )
+    (property "Footprint" "" (id 2) (at 56.896 188.214 0)
+      (effects (font (size 1.27 1.27)) hide)
+    )
+    (property "Datasheet" "~" (id 3) (at 56.896 188.214 0)
       (effects (font (size 1.27 1.27)) hide)
     )
@@
     (pin "9")
   )
+  (symbol (lib_id "Mechanical:MountingHole_Pad") (at 30.734 188.214 180) (unit 1)
+    (in_bom yes) (on_board yes) (fields_autoplaced)
+    (property "Reference" "H5" (id 0) (at 33.274 188.6493 0)
+      (effects (font (size 1.27 1.27)) (justify right))
+    )
+    (property "Value" "" (id 1) (at 33.274 191.1862 0)
+      (effects (font (size 1.27 1.27)) (justify right))
+    )
+    (property "Footprint" "" (id 2) (at 30.734 188.214 0)
+      (effects (font (size 1.27 1.27)) hide)
+    )
+    (property "Datasheet" "~" (id 3) (at 30.734 188.214 0)
+      (effects (font (size 1.27 1.27)) hide)
+    )
+    (pin "1")
+  )
   (sheet (at 196.85 58.42) (size 17.78 15.24) (fields_autoplaced)
     (stroke (width 0) (type solid) (color 0 0 0 0))
@@
       (reference "H4") (unit 1) (value "M3 MountingHole") (footprint "MountingHole:MountingHole_3.2mm_M3_Pad_TopBottom")
     )
+    (path "/e2193abc-3872-42f6-b233-ce70d0a8d732"
+      (reference "H5") (unit 1) (value "POGO_USBDM") (footprint "Stuart_BESPOKE:POGO_D3.50mm_Drill0.9mm")
+    )
+    (path "/53d3f0a5-c8f1-4846-bb9c-97b3d4c70585"
+      (reference "H6") (unit 1) (value "PPOGO_USBDP") (footprint "Stuart_BESPOKE:POGO_D3.50mm_Drill0.9mm")
+    )
     (path "/00000000-0000-0000-0000-00006243dd0b/315ed40d-2ed2-43d4-ab56-86ff969d4795"

Commit message: layout updates
Parts:
- H5: value (none) -> POGO_USBDM; footprint (none) -> Stuart_BESPOKE:POGO_D3.50mm_Drill0.9mm
- H6: value (none) -> PPOGO_USBDP; footprint (none) -> Stuart_BESPOKE:POGO_D3.50mm_Drill0.9mm
- IC4: value (none) -> Raspberry_Pi_Zero_2_W__v1.0_; footprint (none) -> Stuart_BESPOKE:RASPBERRYPIZERO2WV1
- J31: value (none) -> Conn_02x20_Odd_Even_MountingPin; footprint (none) -> Connector_PinHeader_2.54mm:PinHeader_2x20_P2.54mm_Vertical
Other:
- title: The Owl - RPI Cape 16ch Pixel Controller -> RPI Cape DPI 24ch Pixel Controller
Changed lines of the file:
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@@
   (paper "A4")
   (title_block
-    (title "The Owl - RPI Cape 16ch Pixel Controller")
+    (title "RPI Cape DPI 24ch Pixel Controller")
     (date "2022-04-04")
     (company "OnlineDynamic")
@@
     (in_bom yes) (on_board yes)
     (property "Reference" "J31" (id 0) (at 46.99 32.5882 0))
-    (property "Value" "" (id 1) (at 46.99 34.8996 0))
-    (property "Footprint" "" (id 2) (at 45.72 60.96 0)
+    (property "Value" "Conn_02x20_Odd_Even_MountingPin" (id 1) (at 46.99 34.8996 0))
+    (property "Footprint" "Connector_PinHeader_2.54mm:PinHeader_2x20_P2.54mm_Vertical" (id 2) (at 45.72 60.96 0)
       (effects (font (size 1.27 1.27)) hide)
     )
@@
       (effects (font (size 1.27 1.27)) (justify right))
     )
-    (property "Value" "" (id 1) (at 59.436 191.1862 0)
+    (property "Value" "PPOGO_USBDP" (id 1) (at 59.436 191.1862 0)
       (effects (font (size 1.27 1.27)) (justify right))
     )
-    (property "Footprint" "" (id 2) (at 56.896 188.214 0)
+    (property "Footprint" "Stuart_BESPOKE:POGO_D3.50mm_Drill0.9mm" (id 2) (at 56.896 188.214 0)
       (effects (font (size 1.27 1.27)) hide)
     )
@@
     (in_bom yes) (on_board yes)
     (property "Reference" "IC4" (id 0) (at 141.986 29.464 0))
-    (property "Value" "" (id 1) (at 138.43 34.036 0))
-    (property "Footprint" "" (id 2) (at 123.952 20.574 0)
+    (property "Value" "Raspberry_Pi_Zero_2_W__v1.0_" (id 1) (at 138.43 34.036 0))
+    (property "Footprint" "Stuart_BESPOKE:RASPBERRYPIZERO2WV1" (id 2) (at 123.952 20.574 0)
       (effects (font (size 1.27 1.27)) (justify left) hide)
     )
@@
       (effects (font (size 1.27 1.27)) (justify right))
     )
-    (property "Value" "" (id 1) (at 33.274 191.1862 0)
+    (property "Value" "POGO_USBDM" (id 1) (at 33.274 191.1862 0)
       (effects (font (size 1.27 1.27)) (justify right))
     )
-    (property "Footprint" "" (id 2) (at 30.734 188.214 0)
+    (property "Footprint" "Stuart_BESPOKE:POGO_D3.50mm_Drill0.9mm" (id 2) (at 30.734 188.214 0)
       (effects (font (size 1.27 1.27)) hide)
     )
@@
     )
   )
-  (sheet (at 257.81 25.4) (size 19.05 15.24) (fields_autoplaced)
+  (sheet (at 229.362 87.884) (size 19.05 15.24) (fields_autoplaced)
     (stroke (width 0) (type solid) (color 0 0 0 0))
     (fill (color 0 0 0 0.0000))
-    (property "Sheet name" "power" (id 0) (at 257.81 24.6884 0)
+    (property "Sheet name" "power" (id 0) (at 229.362 87.1724 0)
       (effects (font (size 1.27 1.27)) (justify left bottom))
     )
-    (property "Sheet file" "power.kicad_sch" (id 1) (at 257.81 41.2246 0)
+    (property "Sheet file" "power.kicad_sch" (id 1) (at 229.362 103.7086 0)
       (effects (font (size 1.27 1.27)) (justify left top))
     )
@@
     )
   )
-  (sheet (at 201.676 119.634) (size 22.86 16.256) (fields_autoplaced)
+  (sheet (at 256.286 24.384) (size 22.86 16.256) (fields_autoplaced)
     (stroke (width 0.1524) (type solid) (color 0 0 0 0))
     (fill (color 0 0 0 0.0000))
-    (property "Sheet name" "outputs 17-24" (id 0) (at 201.676 118.9224 0)
+    (property "Sheet name" "outputs 17-24" (id 0) (at 256.286 23.6724 0)
       (effects (font (size 1.27 1.27)) (justify left bottom))
     )
-    (property "Sheet file" "outports17-24.kicad_sch" (id 1) (at 201.676 136.4746 0)
+    (property "Sheet file" "outports17-24.kicad_sch" (id 1) (at 256.286 41.2246 0)
       (effects (font (size 1.27 1.27)) (justify left top))
     )
@@
       (reference "#PWR013") (unit 1) (value "GND") (footprint "")
     )
+    (path "/0ef095a5-5266-4228-9874-aea47f1a0c73/aed09ff2-8cdb-4ec1-b27f-d13ddd423151"
+      (reference "#PWR014") (unit 1) (value "+5V") (footprint "")
+    )
     (path "/0ef095a5-5266-4228-9874-aea47f1a0c73/882f1959-4a15-435b-87de-be468139ebfc"
       (reference "#PWR015") (unit 1) (value "+3.3V") (footprint "")
@@
       (reference "#PWR033") (unit 1) (value "GND") (footprint "")
     )
+    (path "/0ef095a5-5266-4228-9874-aea47f1a0c73/5a4c192d-8d3a-40db-ad38-d9db4a269560"
+      (reference "#PWR034") (unit 1) (value "GND") (footprint "")
+    )
+    (path "/0ef095a5-5266-4228-9874-aea47f1a0c73/5d2b0ae3-215c-4435-a957-64088f6e535d"
+      (reference "#PWR035") (unit 1) (value "GND") (footprint "")
+    )
     (path "/00000000-0000-0000-0000-00006235d74f/71bb36b7-6b15-4143-b770-70899c8718b2"
       (reference "#PWR036") (unit 1) (value "GND") (footprint "")
@@
     )
     (path "/00000000-0000-0000-0000-00006243dd0b/00000000-0000-0000-0000-00006264aa53"
-      (reference "C1") (unit 1) (value "0.1uF") (footprint "Capacitor_SMD:CP_Elec_4x5.3")
+      (reference "C1") (unit 1) (value "0.1uF") (footprint "Capacitor_THT:C_Radial_D5.0mm_H11.0mm_P2.00mm")
     )
     (path "/00000000-0000-0000-0000-00006235185d/c446ea81-52d3-45cd-987a-588172881194"
-      (reference "C2") (unit 1) (value "0.1uF") (footprint "3544again:C_0805_2012Metric")
+      (reference "C2") (unit 1) (value "0.1uF") (footprint "Capacitor_THT:C_Radial_D5.0mm_H11.0mm_P2.00mm")
     )
     (path "/00000000-0000-0000-0000-00006256a6bf/8f565d12-9e5c-4925-9ba5-8390f9472918"
-      (reference "C3") (unit 1) (value "0.1uF") (footprint "Capacitor_SMD:CP_Elec_4x5.3")
+      (reference "C3") (unit 1) (value "0.1uF") (footprint "Capacitor_THT:C_Radial_D5.0mm_H11.0mm_P2.00mm")
     )
     (path "/4d354041-9d51-46f1-a4f1-c4cb6a6b9fd8/00000000-0000-0000-0000-000062393073"
-      (reference "C4") (unit 1) (value "0.1uF") (footprint "Capacitor_SMD:CP_Elec_4x5.3")
+      (reference "C4") (unit 1) (value "0.1uF") (footprint "Capacitor_THT:C_Radial_D5.0mm_H11.0mm_P2.00mm")
     )
     (path "/00000000-0000-0000-0000-00006243dd0b/00000000-0000-0000-0000-000062448d86"
@@
       (reference "J32") (unit 1) (value "OLED") (footprint "Connector_PinSocket_2.54mm:PinSocket_1x04_P2.54mm_Vertical")
     )
+    (path "/0ef095a5-5266-4228-9874-aea47f1a0c73/6336394d-7e46-45c7-b073-13cf1cd71142"
+      (reference "J33") (unit 1) (value "GPIO TRG") (footprint "Connector_JST:JST_XH_B3B-XH-A_1x03_P2.50mm_Vertical")
+    )
     (path "/00000000-0000-0000-0000-00006235185d/00000000-0000-0000-0000-0000623a65e4"
       (reference "Q1") (unit 1) (value "MMDT5401") (footprint "Package_TO_SOT_SMD:SOT-363_SC-70-6")
@@
       (reference "R29") (unit 1) (value "4.7k") (footprint "Resistor_SMD:R_0805_2012Metric")
     )
+    (path "/0ef095a5-5266-4228-9874-aea47f1a0c73/306cca96-9f05-42f7-aa13-45be06abf850"
+      (reference "R30") (unit 1) (value "Pull_Up_resistor") (footprint "Resistor_SMD:R_0805_2012Metric")
+    )
+    (path "/0ef095a5-5266-4228-9874-aea47f1a0c73/24e0d778-e59a-460f-afdb-3c30ce14b0a2"
+      (reference "R31") (unit 1) (value "2.2K") (footprint "Resistor_SMD:R_0805_2012Metric")
+    )
+    (path "/0ef095a5-5266-4228-9874-aea47f1a0c73/29607632-33e3-48e1-9775-3167eb70eed8"
+      (reference "R32") (unit 1) (value "2.2K") (footprint "Resistor_SMD:R_0805_2012Metric")
+    )
+    (path "/0ef095a5-5266-4228-9874-aea47f1a0c73/b3a16068-87e8-4a8b-90d6-c7b629d01d49"
+      (reference "R33") (unit 1) (value "2.2K") (footprint "Resistor_SMD:R_0805_2012Metric")
+    )
+    (path "/0ef095a5-5266-4228-9874-aea47f1a0c73/ce709037-b944-48f8-8c08-034461b9727f"
+      (reference "R34") (unit 1) (value "2.2K") (footprint "Resistor_SMD:R_0805_2012Metric")
+    )
     (path "/00000000-0000-0000-0000-00006235185d/00000000-0000-0000-0000-000062380363"
       (reference "R35") (unit 1) (value "10k") (footprint "Resistor_SMD:R_0805_2012Metric")
@@
       (reference "R39") (unit 1) (value "4.7k") (footprint "Resistor_SMD:R_0805_2012Metric")
     )
+    (path "/0ef095a5-5266-4228-9874-aea47f1a0c73/f733e016-a050-4ad2-8a14-7ee1d7da5f26"
+      (reference "R40") (unit 1) (value "2.2K") (footprint "Resistor_SMD:R_0805_2012Metric")
+    )
     (path "/6ac54db5-61c5-4b14-9632-5c95a8268679/cdd226d4-1d4a-4e80-982e-4ec9eeea3d0f"
       (reference "R46") (unit 1) (value "12k") (footprint "Resistor_SMD:R_0805_2012Metric")
@@
       (reference "RN6") (unit 4) (value "33R") (footprint "Resistor_THT:R_Array_SIP8")
     )
+    (path "/0ef095a5-5266-4228-9874-aea47f1a0c73/8076fc12-03a8-4a06-95a1-baaa5e5bcd6c"
+      (reference "SW1") (unit 1) (value "SW_UP") (footprint "Button_Switch_THT:SW_PUSH_6mm")
+    )
+    (path "/0ef095a5-5266-4228-9874-aea47f1a0c73/b035374f-1a0b-45b9-a281-2ea2a5d3e5aa"
+      (reference "SW2") (unit 1) (value "SW_DOWN") (footprint "Button_Switch_THT:SW_PUSH_6mm")
+    )
+    (path "/0ef095a5-5266-4228-9874-aea47f1a0c73/a6a47508-8877-4ab7-828f-fbfd1a8194aa"
+      (reference "SW3") (unit 1) (value "SW_BACK") (footprint "Button_Switch_THT:SW_PUSH_6mm")
+    )
+    (path "/0ef095a5-5266-4228-9874-aea47f1a0c73/55e4a9f4-3e09-4d75-ad4c-618e19e6d599"
+      (reference "SW4") (unit 1) (value "SW_TEST") (footprint "Button_Switch_THT:SW_PUSH_6mm")
+    )
+    (path "/0ef095a5-5266-4228-9874-aea47f1a0c73/e1308ef9-4b3c-46aa-a949-80a51e780b05"
+      (reference "SW5") (unit 1) (value "SW_ENTER") (footprint "Button_Switch_THT:SW_PUSH_6mm")
+    )
     (path "/00000000-0000-0000-0000-00006235185d/00000000-0000-0000-0000-00006237f70d"
-      (reference "U1") (unit 1) (value "AT24C256C") (footprint "Package_SO:SOIC-8_3.9x4.9mm_P1.27mm")
+      (reference "U1") (unit 1) (value "AT24C256C") (footprint "Package_DIP:DIP-8_W7.62mm_Socket")
     )
     (path "/00000000-0000-0000-0000-00006235d74f/468a6ca1-df23-470b-b627-0cc0221c989b"

Commit message: more layout tweaking and a bit of copper!
Connections:
- net DATA10: now also J31.35 (Pin_35); no longer J31.33 (Pin_33)
- net DATA11: now also J31.33 (Pin_33); no longer J31.35 (Pin_35)
- net DATA12: now also J31.31 (Pin_31); no longer J31.37 (Pin_37)
- net DATA9: now also J31.37 (Pin_37); no longer J31.31 (Pin_31)
- net USBDM: no longer IC4.49 (USB_DM)
- net USBDP: no longer IC4.48 (USB_DP)
- no-connect marks 61 -> 63
Other:
- note added: "can they GPIO EEPROMPINS be used for triggers for switch and ext trigger?"
Changed lines of the file:
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@@
   (no_connect (at 177.292 75.184))
   (no_connect (at 177.292 114.554))
+  (no_connect (at 87.122 164.338))
+  (no_connect (at 92.202 164.338))
   (no_connect (at 104.902 81.534))
   (no_connect (at 104.902 99.314))
@@
     (stroke (width 0) (type default) (color 0 0 0 0))
   )
+  (text "can they GPIO EEPROMPINS be used for triggers for switch and ext trigger?"
+    (at 15.494 93.472 0)
+    (effects (font (size 1.27 1.27)) (justify left bottom))
+  )
   (text "DPI-24" (at 220.98 157.48 0)
     (effects (font (size 8.001 8.001) italic) (justify left bottom))
@@
     )
   )
-  (global_label "USBDP" (shape bidirectional) (at 87.122 164.338 270) (fields_autoplaced)
-    (effects (font (size 1.27 1.27)) (justify right))
-    (property "Intersheet References" "${INTERSHEET_REFS}" (id 0) (at 87.0426 173.0122 90)
-      (effects (font (size 1.27 1.27)) (justify right) hide)
-    )
-  )
-  (global_label "DATA10" (shape output) (at 36.83 78.74 180) (fields_autoplaced)
+  (global_label "DATA11" (shape output) (at 36.83 78.74 180) (fields_autoplaced)
     (effects (font (size 1.27 1.27)) (justify right))
     (property "Intersheet References" "${INTERSHEET_REFS}" (id 0) (at 27.672 78.6606 0)
@@
     )
   )
-  (global_label "DATA12" (shape output) (at 36.83 83.82 180) (fields_autoplaced)
+  (global_label "DATA9" (shape output) (at 36.83 83.82 180) (fields_autoplaced)
     (effects (font (size 1.27 1.27)) (justify right))
-    (property "Intersheet References" "${INTERSHEET_REFS}" (id 0) (at 27.672 83.7406 0)
+    (property "Intersheet References" "${INTERSHEET_REFS}" (id 0) (at 28.8815 83.7406 0)
       (effects (font (size 1.27 1.27)) (justify right) hide)
     )
@@
     )
   )
-  (global_label "DATA9" (shape output) (at 36.83 76.2 180) (fields_autoplaced)
+  (global_label "DATA12" (shape output) (at 36.83 76.2 180) (fields_autoplaced)
     (effects (font (size 1.27 1.27)) (justify right))
-    (property "Intersheet References" "${INTERSHEET_REFS}" (id 0) (at 28.8815 76.1206 0)
+    (property "Intersheet References" "${INTERSHEET_REFS}" (id 0) (at 27.672 76.1206 0)
       (effects (font (size 1.27 1.27)) (justify right) hide)
     )
@@
     )
   )
-  (global_label "USBDM" (shape bidirectional) (at 92.202 164.338 270) (fields_autoplaced)
-    (effects (font (size 1.27 1.27)) (justify right))
-    (property "Intersheet References" "${INTERSHEET_REFS}" (id 0) (at 92.1226 173.1936 90)
-      (effects (font (size 1.27 1.27)) (justify right) hide)
-    )
-  )
   (global_label "DATA3" (shape output) (at 36.83 53.34 180) (fields_autoplaced)
     (effects (font (size 1.27 1.27)) (justify right))
@@
     )
   )
-  (global_label "DATA11" (shape output) (at 36.83 81.28 180) (fields_autoplaced)
+  (global_label "DATA10" (shape output) (at 36.83 81.28 180) (fields_autoplaced)
     (effects (font (size 1.27 1.27)) (justify right))
     (property "Intersheet References" "${INTERSHEET_REFS}" (id 0) (at 27.672 81.2006 0)
@@
       (reference "#PWR0159") (unit 1) (value "GND") (footprint "")
     )
+    (path "/00000000-0000-0000-0000-00006235d74f/da59ff4d-eb84-4ab6-a0c6-20d1e800afb6"
+      (reference "#PWR0160") (unit 1) (value "GND") (footprint "")
+    )
+    (path "/0ef095a5-5266-4228-9874-aea47f1a0c73/1d1a9038-8e2a-49c4-ae48-664a7e20b7f4"
+      (reference "#PWR0161") (unit 1) (value "GND") (footprint "")
+    )
+    (path "/0ef095a5-5266-4228-9874-aea47f1a0c73/7f2af5c3-8684-4ba1-a454-5d9fb05972cc"
+      (reference "#PWR0162") (unit 1) (value "GND") (footprint "")
+    )
+    (path "/0ef095a5-5266-4228-9874-aea47f1a0c73/b4d20fc8-ddb5-4660-a4ed-c05cfdce7f5f"
+      (reference "#PWR0163") (unit 1) (value "GND") (footprint "")
+    )
+    (path "/0ef095a5-5266-4228-9874-aea47f1a0c73/84a85c9d-1a7d-41fd-a30b-4226cce52ad3"
+      (reference "#PWR0164") (unit 1) (value "+5V") (footprint "")
+    )
     (path "/00000000-0000-0000-0000-00006243dd0b/00000000-0000-0000-0000-00006264aa53"
       (reference "C1") (unit 1) (value "0.1uF") (footprint "Capacitor_THT:C_Radial_D5.0mm_H11.0mm_P2.00mm")
@@
       (reference "C4") (unit 1) (value "0.1uF") (footprint "Capacitor_THT:C_Radial_D5.0mm_H11.0mm_P2.00mm")
     )
+    (path "/0ef095a5-5266-4228-9874-aea47f1a0c73/05263be5-e9a4-4427-af9e-fbcdb83808e2"
+      (reference "C5") (unit 1) (value "0.1uF") (footprint "Capacitor_THT:C_Radial_D5.0mm_H11.0mm_P2.00mm")
+    )
     (path "/00000000-0000-0000-0000-00006243dd0b/00000000-0000-0000-0000-000062448d86"
       (reference "D1") (unit 1) (value "0603") (footprint "LED_SMD:LED_0603_1608Metric")
@@
       (reference "J33") (unit 1) (value "GPIO TRG") (footprint "Connector_JST:JST_XH_B3B-XH-A_1x03_P2.50mm_Vertical")
     )
+    (path "/00000000-0000-0000-0000-00006235d74f/9519f722-c928-4685-9aab-2867fdd8d1de"
+      (reference "J34") (unit 1) (value "Select Voltage") (footprint "Connector_PinHeader_2.54mm:PinHeader_1x03_P2.54mm_Vertical")
+    )
+    (path "/00000000-0000-0000-0000-00006235d74f/b22242e4-117b-4904-89f4-7246dcb75328"
+      (reference "J35") (unit 1) (value "Select Control Feed") (footprint "Connector_PinHeader_2.54mm:PinHeader_1x03_P2.54mm_Vertical")
+    )
+    (path "/00000000-0000-0000-0000-00006235d74f/c075caff-ca37-4800-b0e4-31bd6f4d253c"
+      (reference "J36") (unit 1) (value "Aux In") (footprint "TerminalBlock_RND:TerminalBlock_RND_205-00012_1x02_P5.00mm_Horizontal")
+    )
     (path "/00000000-0000-0000-0000-00006235185d/00000000-0000-0000-0000-0000623a65e4"
       (reference "Q1") (unit 1) (value "MMDT5401") (footprint "Package_TO_SOT_SMD:SOT-363_SC-70-6")
@@
       (reference "U4") (unit 2) (value "LAN7500-ABJZ") (footprint "Package_DFN_QFN:QFN-56-1EP_8x8mm_P0.5mm_EP5.9x5.9mm")
     )
-  )
+    (path "/0ef095a5-5266-4228-9874-aea47f1a0c73/bfcea11a-f536-4ff2-a606-a279cb227a21"
+      (reference "U5") (unit 1) (value "ADS1113IDGS") (footprint "Package_SO:TSSOP-10_3x3mm_P0.5mm")
+    )
+  )
