File: KiCAD/DPI-24/DPI-24-Controller/DPI-24-Controller.kicad_pcb (KiCad board)
At the start: 2 copper layers, 230 x 120 mm, 155 parts, among them IC1 SN74AHC245N, IC2 SN74AHC245N, IC3 SN74AHC245N, IC4 Raspberry_Pi_Zero_2_W__v1.0_, IC5 KSZ8794CNXIC, J1 G D V, J10 G D V, J11 G D V, J12 G D V, J13 G D V, J14 G D V, J15 G D V, J16 G D V, J17 G D V, J18 G D V, J19 G D V, J2 G D V, J20 G D V, J21 G D V, J22 G D V, J23 G D V, J24 G D V, J25 UPLINK, J26 LAN 1, J27 LAN 2, J28 1-8 In, J29 9-16 In, J3 G D V, J30 17-24 In, J31 Conn_02x20_Odd_Even_MountingP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, J32 OLED, J4 G D V, J5 G D V, J6 G D V, J7 G D V, J8 G D V, J9 G D V, Q1 MMDT5401, Q2 DMG2302U, U1 AT24C256C, U2 D-SUN_MP1584_BUCK, U3 TZT_Original_0.96_inch_oled_I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, U4 LAN7500-ABJZ

Commit message: dpi-24 updates
Parts:
- added H5: POGO_USBDM, Stuart_BESPOKE:POGO_D3.50mm_Drill0.9mm, F.Cu at (130.8, 78.3)
- added H6: PPOGO_USBDP, Stuart_BESPOKE:POGO_D3.50mm_Drill0.9mm, F.Cu at (129.4, 81.9)
- moved J30 10.1 mm to (264.8, 138.3), turned to 90 degrees
- moved C4 3.92 mm to (209.9, 58.4)
- moved J17 2.65 mm to (230.1, 116.2)
- moved J19 2.65 mm to (230.1, 98.0)
- moved J21 2.65 mm to (230.1, 79.8)
- moved J23 2.65 mm to (230.1, 61.6)
- moved RN5 2.65 mm to (218.6, 102.0)
- moved RN6 2.65 mm to (218.8, 75.7)

Commit message: layout updates
Parts:
- added J33: GPIO TRG, Connector_JST:JST_XH_B3B-XH-A_1x03_P2.50mm_Vertical, F.Cu at (49.7, 58.0)
- added R30: Pull_Up_resistor, Resistor_SMD:R_0805_2012Metric, F.Cu at (157.6, 47.6)
- added R31: 2.2K, Resistor_SMD:R_0805_2012Metric, F.Cu at (177.2, 46.2)
- added R32: 2.2K, Resistor_SMD:R_0805_2012Metric, F.Cu at (177.1, 50.2)
- added R33: 2.2K, Resistor_SMD:R_0805_2012Metric, F.Cu at (176.9, 54.2)
- added R34: 2.2K, Resistor_SMD:R_0805_2012Metric, F.Cu at (176.9, 58.0)
- added R40: 2.2K, Resistor_SMD:R_0805_2012Metric, F.Cu at (177.0, 60.6)
- added SW1: SW_UP, Button_Switch_THT:SW_PUSH_6mm, F.Cu at (199.2, 40.2)
- added SW2: SW_DOWN, Button_Switch_THT:SW_PUSH_6mm, F.Cu at (199.5, 56.5)
- added SW3: SW_BACK, Button_Switch_THT:SW_PUSH_6mm, F.Cu at (188.5, 48.4)
- added SW4: SW_TEST, Button_Switch_THT:SW_PUSH_6mm, F.Cu at (160.6, 71.1)
- added SW5: SW_ENTER, Button_Switch_THT:SW_PUSH_6mm, F.Cu at (210.1, 48.4)
- C1, C2, C3, C4: footprint Capacitor_SMD:CP_Elec_4x5.3 -> Capacitor_THT:C_Radial_D5.0mm_H11.0mm_P2.00mm
- U1: footprint Package_SO:SOIC-8_3.9x4.9mm_P1.27mm -> Package_DIP:DIP-8_W7.62mm_Socket
- moved C2 75.7 mm to (191.3, 73.0), turned to -90 degrees
- moved U1 66.7 mm to (177.1, 72.4)
- moved R28 56.1 mm to (127.0, 62.5)
- moved R29 56.1 mm to (127.0, 65.4)
- moved D33 46.5 mm to (121.7, 57.6)
- moved D34 46.5 mm to (121.7, 60.1)
- moved C3 32.1 mm to (195.2, 87.8)
- moved R46 22.1 mm to (100.6, 68.2)
- moved F28 19.5 mm to (65.7, 83.8), turned to 180 degrees
- moved R35 18.5 mm to (73.7, 67.2)
- moved R47 18.1 mm to (100.4, 72.1)
- moved R36 16.5 mm to (68.7, 67.1)
- moved C4 12.3 mm to (213.6, 70.1), turned to -90 degrees
- moved Q1 11.2 mm to (68.6, 72.9)
- moved Q2 11.2 mm to (73.9, 73.1)
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
Commit message: pcb layout changes
Parts:
- J28: value 1-8 In -> 1-8 In 12V DC
- J29: value 9-16 In -> 9-16 In 12V DC
- J30: value 17-24 In -> 17-24 In 12V DC
- moved D32 12.5 mm to (58.2, 75.6), turned to 180 degrees
- moved R39 10.9 mm to (63.0, 77.0), turned to 90 degrees
- moved D1 5.33 mm to (75.6, 137.6)
- moved D31 5.14 mm to (62.8, 72.3)
- moved D30 3.11 mm to (251.8, 125.1)
- moved D28 2.40 mm to (239.1, 133.2)
- moved RN5 2.34 mm to (220.9, 101.8)
- moved RN6 2.34 mm to (221.1, 75.4)
- moved F26 2.22 mm to (228.4, 150.1)
- moved D25 2.19 mm to (63.7, 150.3)
- moved R1 2.03 mm to (75.6, 141.1), turned to 90 degrees
- moved R37 1.90 mm to (63.6, 146.3), turned to -90 degrees
- moved D7 1.80 mm to (134.6, 137.7), turned to -90 degrees
- moved D4 1.60 mm to (105.1, 137.7), turned to -90 degrees
- moved D8 1.59 mm to (144.6, 137.7), turned to -90 degrees
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
Commit message: further layout updates
Parts:
- J28: value 1-8 In 12V DC -> Ports 1-8 12V DC IN; footprint TerminalBlock_MetzConnect:TerminalBlock_MetzConnect_Type703_RT10N02HGLU_1x02_P9.52mm_Horizontal -> Stuart_BESPOKE:TerminalBlock_KF950_1x02_P9.50mm_Horizontal
- J29: value 9-16 In 12V DC -> Ports 9-16 12V DC IN; footprint TerminalBlock_MetzConnect:TerminalBlock_MetzConnect_Type703_RT10N02HGLU_1x02_P9.52mm_Horizontal -> Stuart_BESPOKE:TerminalBlock_KF950_1x02_P9.50mm_Horizontal
- J30: value 17-24 In 12V DC -> Ports 17-24 12V DC IN; footprint TerminalBlock_MetzConnect:TerminalBlock_MetzConnect_Type703_RT10N02HGLU_1x02_P9.52mm_Horizontal -> Stuart_BESPOKE:TerminalBlock_KF950_1x02_P9.50mm_Horizontal
- SW1: value SW_UP -> UP
- SW2: value SW_DOWN -> DOWN
- SW3: value SW_BACK -> BACK
- SW4: value SW_TEST -> TEST
- SW5: value SW_ENTER -> ENTER
- moved J28 15.7 mm to (46.7, 114.5), turned to -90 degrees
- moved J29 15.3 mm to (237.3, 153.8), turned to 0 degrees
- moved J30 9.44 mm to (272.7, 143.5)
- moved J33 6.51 mm to (50.3, 64.5)
- moved D26 1.10 mm to (64.7, 135.6)
Connections:
- J28 pad 1: GND -> V1
- J28 pad 2: V1 -> GND
- J30 pad 1: GND -> V3
- J30 pad 2: V3 -> GND
Other:
- board text added: "OLED MENU"

Commit message: more layout tweaking and a bit of copper!
Parts:
- removed J33: GPIO TRG, Connector_JST:JST_XH_B3B-XH-A_1x03_P2.50mm_Vertical
- added ?: , clipboard:25d1d928-aa0c-4bb1-b9d4-6d036955ffcd, F.Cu at (159.1, 105.0)
- added C5: 0.1uF, Capacitor_THT:C_Radial_D5.0mm_H11.0mm_P2.00mm, F.Cu at (189.1, 61.0)
- added J34: Select Voltage, Connector_PinHeader_2.54mm:PinHeader_1x03_P2.54mm_Vertical, F.Cu at (56.6, 96.9)
- added J35: Select Control Feed, Connector_PinHeader_2.54mm:PinHeader_1x03_P2.54mm_Vertical, F.Cu at (58.9, 104.4)
- added J36: Aux In, TerminalBlock_RND:TerminalBlock_RND_205-00012_1x02_P5.00mm_Horizontal, F.Cu at (52.0, 109.4)
- added U5: ADS1113IDGS, Package_SO:TSSOP-10_3x3mm_P0.5mm, F.Cu at (181.5, 45.9)
- moved C2 81.0 mm to (112.1, 89.8)
- moved IC4 71.3 mm to (123.4, -31.9)
- moved U1 62.4 mm to (117.3, 90.0)
- moved D29 27.3 mm to (244.7, 117.7)
- moved R26 27.3 mm to (244.5, 113.8)
- moved R17 24.0 mm to (234.7, 113.4), turned to -90 degrees
- moved R9 23.4 mm to (153.9, 118.9), turned to 180 degrees
- moved R21 23.3 mm to (234.9, 75.8), turned to -90 degrees
- moved R23 23.2 mm to (234.8, 56.8), turned to -90 degrees
- moved R19 23.2 mm to (234.9, 94.6), turned to -90 degrees
- moved R13 23.1 mm to (194.1, 119.3), turned to 180 degrees
- moved R7 23.0 mm to (133.8, 119.1), turned to 180 degrees
- moved R15 22.7 mm to (210.8, 119.3), turned to 180 degrees
- moved R11 22.7 mm to (173.7, 119.3), turned to 180 degrees
- moved R5 22.6 mm to (113.7, 119.0), turned to 180 degrees
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Connections:
- IC4 pad 48: USBDP -> unconnected-(IC4-Pad48)
- IC4 pad 49: USBDM -> unconnected-(IC4-Pad49)
- J31 pad 31: DATA9 -> DATA12
- J31 pad 33: DATA10 -> DATA11
- J31 pad 35: DATA11 -> DATA10
- J31 pad 37: DATA12 -> DATA9
- U2 pad 2: unconnected-(U2-Pad2) -> GND
- U2 pad 3: VIN1 -> BUCK_In
- U2 pad 4: unconnected-(U2-Pad4) -> BUCK_In
- U2 pad 6: unconnected-(U2-Pad6) -> GND1
- U2 pad 8: unconnected-(U2-Pad8) -> V5
Routing:
- net DATA1: track 0.00 -> 94.8 mm
- net DATA2: track 0.00 -> 90.2 mm
- net DATA3: track 0.00 -> 86.6 mm
- net DATA4: track 0.00 -> 83.0 mm
- net +5V: track 0.00 -> 82.1 mm
- net DATA24: track 0.00 -> 72.6 mm
- net DATA5: track 0.00 -> 71.9 mm
- net DATA21: track 0.00 -> 70.6 mm
- net DATA23: track 0.00 -> 70.5 mm
- net DATA22: track 0.00 -> 68.5 mm
- net DATA6: track 0.00 -> 67.6 mm
- net DATA7: track 0.00 -> 64.0 mm
- net DATA20: track 0.00 -> 62.4 mm
- net DATA19: track 0.00 -> 58.7 mm
- net DATA8: track 0.00 -> 58.5 mm
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- added copper zone on F.Cu, net Net-(F1-Pad3)
- added copper zone on F.Cu, net Net-(F10-Pad3)
- added copper zone on F.Cu, net Net-(F11-Pad3)
- added copper zone on F.Cu, net Net-(F12-Pad3)
- added copper zone on F.Cu, net Net-(F13-Pad3)
- added copper zone on F.Cu, net Net-(F14-Pad3)
- added copper zone on F.Cu, net Net-(F15-Pad3)
- added copper zone on F.Cu, net Net-(F16-Pad3)
- added copper zone on F.Cu, net Net-(F2-Pad3)
- added copper zone on F.Cu, net Net-(F3-Pad3)
- added copper zone on F.Cu, net Net-(F4-Pad3)
- added copper zone on F.Cu, net Net-(F5-Pad3)
- added copper zone on F.Cu, net Net-(F6-Pad3)
- added copper zone on F.Cu, net Net-(F7-Pad3)
- added copper zone on F.Cu, net Net-(F8-Pad3)
- added copper zone on F.Cu, net Net-(F9-Pad3)
- added copper zone on B.Cu, net V1
- added copper zone on F.Cu, net V1
- added copper zone on B.Cu, net V2
- added copper zone on F.Cu, net V2
- added copper zone on B.Cu, net V3
- added copper zone on F.Cu, net V3
- added copper zone on B.Cu, net VIN1
- added copper zone on F.Cu, net VIN1
- added copper zone on B.Cu, net VIN2
- added copper zone on F.Cu, net VIN2
- added copper zone on B.Cu, net VIN3
- added copper zone on F.Cu, net VIN3
Other:
- board text added: "+DC"
- board text added: "12V"
- board text added: "5V"
- board text added: "AUX"
- board text added: "EEPROM"
- board text added: "GND"
- board text added: "RASPBERRY PI ZERO 2"
- board text added: "SN74AHC245N"
- board text added: "System Power"
- board text added: "V1"

Commit message: more tweaks
Parts:
- moved Q2 2.03 mm to (76.4, 69.8)
- moved R35 2.03 mm to (76.2, 64.0)
- moved R36 2.03 mm to (71.2, 63.9)
- moved Q1 2.03 mm to (71.1, 69.6)
- moved R26 0.41 mm to (244.0, 113.8), turned to 180 degrees
- moved U3 0.05 mm to (161.3, 37.6)
Routing:
- net +5V: track 82.1 -> 222.8 mm
- net +3V3: track 0.00 -> 54.1 mm, vias 0 -> 2
- net VIN2: track 4.29 -> 40.3 mm
- net VIN3: track 0.00 -> 30.6 mm
- net Net-(D31-Pad2): track 0.00 -> 9.06 mm
- net Net-(D29-Pad2): track 0.00 -> 3.78 mm
- net Net-(F17-Pad3): track 30.4 -> 31.9 mm
